File: VCADSR/VCADSR.kicad_pcb (KiCad board)
At the start: 4 copper layers, 140.2 x 128.5 mm, 107 parts, among them J1 Conn_01x01_Pin, J2 Conn_01x16_Pin, J3 Conn_01x16_Pin, J4 Conn_01x06_Pin, Q1 BC557, Q10 BC547, Q11 BC547, Q12 NMOS, Q13 NMOS, Q14 BC547, Q15 BC547, Q16 BC547, Q17 BC547, Q2 BC557, Q3 BC547, Q4 BC547, Q5 NMOS, Q6 BC547, Q7 BC547, Q8 BC557, Q9 BC557, SW1 SW_Push, U1 TL074, U13 Aux_flush, U14 4066, U15 TL074, U16 Aux_flush, U17 Aux_flush, U19 Aux_flush, U2 Aux_flush, U20 Aux_flush, U3 Aux_flush, U4 Aux_flush, U5 Aux_flush, U6 Switch, U7 Aux_flush, U8 Switch, U9 4001

Commit message: Add files via upload
Updated Files
Parts:
- removed R10, R16, R18, R20: R, Resistor_SMD:R_1206_3216Metric
- moved U19 19.0 mm to (163.9, 136.5), turned to 90 degrees
- moved U20 16.5 mm to (174.7, 136.5), turned to 90 degrees
- moved U17 8.53 mm to (153.1, 136.5), turned to 90 degrees
- moved U16 7.17 mm to (142.3, 136.5), turned to 90 degrees
- moved SW1 4.00 mm to (188.7, 136.5), turned to 90 degrees
- moved R11 3.64 mm to (154.9, 57.6), turned to 180 degrees
- moved R21 1.35 mm to (157.2, 112.9), turned to 180 degrees
- moved D4 0.50 mm to (157.2, 61.9)
- moved D5 0.50 mm to (157.2, 81.0)
- moved D6 0.50 mm to (156.7, 98.8)
- moved D7 0.50 mm to (157.2, 116.5)
- moved R19 0.32 mm to (157.2, 94.9), turned to 180 degrees
- moved R17 0.19 mm to (158.3, 77.1), turned to 180 degrees
Connections:
- D4 pad 1: Net-(D4-K) -> GND
- D5 pad 1: Net-(D5-K) -> GND
- D6 pad 1: Net-(D6-K) -> GND
- D7 pad 1: Net-(D7-K) -> GND
- Q14 pad 1: Net-(D4-K) -> +12V
- Q14 pad 2: Net-(Q14-B) -> APHS
- Q14 pad 3: GND -> Net-(Q14-E)
- Q15 pad 1: Net-(D5-K) -> +12V
- Q15 pad 2: Net-(Q15-B) -> DPHS
- Q15 pad 3: GND -> Net-(Q15-E)
- Q16 pad 1: Net-(D6-K) -> +12V
- Q16 pad 2: Net-(Q16-B) -> SPHS
- Q16 pad 3: GND -> Net-(Q16-E)
- Q17 pad 1: Net-(D7-K) -> +12V
- Q17 pad 2: Net-(Q17-B) -> RPHS
- Q17 pad 3: GND -> Net-(Q17-E)
- R11 pad 2: +12V -> Net-(Q14-E)
- R17 pad 2: +12V -> Net-(Q15-E)
- R19 pad 2: +12V -> Net-(Q16-E)
- R21 pad 2: +12V -> Net-(Q17-E)
Routing:
- net Net-(RV10-Pad1): track 62.0 -> 79.8 mm
- net GND: track 61.0 -> 77.2 mm
- net Net-(RV12-Pad1): track 54.3 -> 70.3 mm
- net Net-(Q14-B): track 13.8 -> 0.00 mm
- net Net-(RV6-Pad1): track 80.4 -> 94.1 mm
- net APHS: track 191.6 -> 178.9 mm
- net Net-(Q15-B): track 11.4 -> 0.00 mm
- net DPHS: track 119.1 -> 129.2 mm
- net +12V: track 50.0 -> 60.1 mm
- net Net-(Q15-E): track 0.00 -> 8.75 mm
- net Net-(RV8-Pad1): track 72.7 -> 81.1 mm
- net Net-(D7-K): track 7.90 -> 0.00 mm
- net Net-(Q16-E): track 0.00 -> 5.50 mm
- net Net-(Q14-E): track 0.00 -> 4.55 mm
- net Net-(D6-K): track 4.54 -> 0.00 mm
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Other:
- board text added: "ATT"
- board text added: "CV:"
- board text added: "DEC"
- board text added: "REL"
- board text added: "SUS"
- board text added: "x4"
- board text removed: "A"
- board text removed: "CV"
- board text removed: "D"
- board text removed: "R"
- board text removed: "S"
- board text removed: "x10"
