File: VCADSR/VCADSR.kicad_sch (KiCad schematic)
At the start: 103 parts, among them J1 Conn_01x01_Pin, J2 Conn_01x16_Pin, J3 Conn_01x16_Pin, J4 Conn_01x06_Pin, Q1 BC557, Q10 BC547, Q11 BC547, Q12 NMOS, Q13 NMOS, Q14 BC547, Q15 BC547, Q16 BC547, Q17 BC547, Q2 BC557, Q3 BC547, Q4 BC547, Q5 NMOS, Q6 BC547, Q7 BC547, Q8 BC557, Q9 BC557, SW1 SW_Push, U1 TL074, U13 Aux_flush, U14 4066, U15 TL074, U16 Aux_flush, U17 Aux_flush, U19 Aux_flush, U2 Aux_flush, U20 Aux_flush, U3 Aux_flush, U4 Aux_flush, U5 Aux_flush, U6 Switch, U7 Aux_flush, U8 Switch, U9 4001

Commit message: Add files via upload
Updated Files
Parts:
- removed R10, R16, R18, R20: R, Resistor_SMD:R_1206_3216Metric, symbol Device:R
Connections:
- net +12V: now also Q14.1 (C), Q15.1 (C), Q16.1 (C), Q17.1 (C); no longer R11.2, R17.2, R19.2, R21.2
- net APHS: now also Q14.2 (B)
- net DPHS: now also Q15.2 (B)
- net GND: now also D4.1 (K), D5.1 (K), D6.1 (K), D7.1 (K); no longer Q14.3 (E), Q15.3 (E), Q16.3 (E), Q17.3 (E)
- net RPHS: now also Q17.2 (B)
- net SPHS: now also Q16.2 (B)
- net ININV: now reaches Q12.2 (G), Q7.1 (C), R39.2, R40.1, U14.12
- new net: Q16.3 (E), R19.2
- new net: Q17.3 (E), R21.2
- new net: Q15.3 (E), R17.2
- new net: Q14.3 (E), R11.2
Other:
- note added: "ADSR Block"
- note added: "CV Summing"
- note added: "LEDs/Stage Outputs"
- note added: "LOOP"
- note added: "Logic"
- note added: "MANUAL"
- note added: "x4"
- moved on the sheet: D4, D5, D6, D7, J1, J2, J3, J4, Q12, Q13, Q5, SW1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
