File: Drum/Drum.kicad_pcb (KiCad board)
At the start: 2 copper layers, 92.1 x 128 mm, 66 parts, among them J1 Conn_01x06_Pin, J2 Conn_01x11_Pin, J3 Conn_01x11_Pin, J4 Conn_01x11_Pin, Q10 BC557, Q2 BC547, Q3 BC547, Q4 BC557, Q5 BC557, Q6 BC547, Q7 BC547, Q8 BC547, Q9 BC547, SW1 SW_SPDT, U1 Aux_flush, U2 Aux_flush, U3 TL074, U5 LM13700, U6 Aux_flush, U7 Aux_flush, U8 Aux_flush

Commit message: Add files via upload
Parts:
- removed J4: Conn_01x11_Pin, Connector_PinHeader_2.54mm:PinHeader_1x01_P2.54mm_Vertical
- removed R26: 1k, Resistor_THT:R_Axial_DIN0207_L6.3mm_D2.5mm_P7.62mm_Horizontal
- added D4: D, Diode_THT:D_A-405_P7.62mm_Horizontal, B.Cu at (124.4, 96.0)
- C1: value 5n -> 10n
- C3: value 5n -> 470nF or omit
- C4: value 5n -> 2 to 10nF
- R15, R28, R31: value 100k -> 47k
- R16, R33: value 100k -> 1k
- R17: value 100k -> 2k2
- R22, R32: value 100k -> 10k
- R24: value 10k -> 100k
Connections:
- U5 pad 4: Net-(U5C--) -> GND
Routing:
- net Net-(U5C-+): track 20.9 -> 12.6 mm
- net Net-(D4-K): track 8.98 -> 16.1 mm
- net Net-(U5C--): track 3.60 -> 0.00 mm
