File: Drum/Drum.kicad_sch (KiCad schematic)
At the start: 62 parts, among them J1 Conn_01x06_Pin, J2 Conn_01x11_Pin, J3 Conn_01x11_Pin, J4 Conn_01x11_Pin, Q10 BC557, Q2 BC547, Q3 BC547, Q4 BC557, Q5 BC557, Q6 BC547, Q7 BC547, Q8 BC547, Q9 BC547, SW1 SW_SPDT, U1 Aux_flush, U2 Aux_flush, U3 TL074, U5 LM13700, U6 Aux_flush, U7 Aux_flush, U8 Aux_flush

Commit message: Add files via upload
Parts:
- removed J4: Conn_01x11_Pin, Connector_PinHeader_2.54mm:PinHeader_1x01_P2.54mm_Vertical, symbol Connector:Conn_01x01_Pin
- removed R26: omit, Resistor_THT:R_Axial_DIN0207_L6.3mm_D2.5mm_P7.62mm_Horizontal, symbol Device:R
- added D4: D, Diode_THT:D_A-405_P7.62mm_Horizontal, symbol Device:D
- C2: value 5n -> 1u to 5u
- R19: value 1k -> 100k
- R33: value 0R -> 1k
Connections:
- net GND: now also U5.4 (-), D4.2 (A)
- net at Q10.2 (B), R33.2: now also D4.1 (K)
Changed lines of the file:
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@@
   (junction (at 99.06 44.45) (diameter 0) (color 0 0 0 0)
   )
+  (junction (at 96.5919 65.278) (diameter 0) (color 0 0 0 0)
+  )
   (junction (at 116.967 170.942) (diameter 0) (color 0 0 0 0)
   )
@@
   (junction (at 186.182 107.188) (diameter 0) (color 0 0 0 0)
   )
-  (junction (at 197.485 45.085) (diameter 0) (color 0 0 0 0)
-  )
   (junction (at 115.316 106.934) (diameter 0) (color 0 0 0 0)
   )
   (junction (at 118.237 174.752) (diameter 0) (color 0 0 0 0)
   )
-  (junction (at 207.518 52.578) (diameter 0) (color 0 0 0 0)
-  )
   (junction (at 93.98 44.45) (diameter 0) (color 0 0 0 0)
   )
@@
     (stroke (width 0) (type default))
   )
+  (wire (pts (xy 197.485 45.085) (xy 210.058 45.085))
+    (stroke (width 0) (type default))
+  )
   (wire (pts (xy 137.414 53.086) (xy 137.414 60.198))
     (stroke (width 0) (type default))
@@
     (stroke (width 0) (type default))
   )
-  (wire (pts (xy 210.058 44.958) (xy 210.058 47.498))
-    (stroke (width 0) (type default))
-  )
   (wire (pts (xy 81.28 22.86) (xy 81.28 34.29))
     (stroke (width 0) (type default))
@@
     (stroke (width 0) (type default))
   )
+  (wire (pts (xy 210.058 45.085) (xy 210.058 47.498))
+    (stroke (width 0) (type default))
+  )
   (wire (pts (xy 60.96 53.34) (xy 60.96 49.53))
     (stroke (width 0) (type default))
@@
     (stroke (width 0) (type default))
   )
-  (wire (pts (xy 206.248 52.578) (xy 207.518 52.578))
-    (stroke (width 0) (type default))
-  )
   (wire (pts (xy 116.967 170.942) (xy 125.857 170.942))
     (stroke (width 0) (type default))
@@
     (stroke (width 0) (type default))
   )
-  (wire (pts (xy 197.485 45.085) (xy 206.375 45.085))
-    (stroke (width 0) (type dash) (color 0 0 194 1))
-  )
   (wire (pts (xy 270.764 75.692) (xy 270.764 74.422))
     (stroke (width 0) (type default))
@@
     (stroke (width 0) (type default))
   )
-  (wire (pts (xy 207.518 44.958) (xy 210.058 44.958))
+  (wire (pts (xy 130.556 118.364) (xy 130.556 109.474))
     (stroke (width 0) (type default))
   )
-  (wire (pts (xy 130.556 118.364) (xy 130.556 109.474))
+  (wire (pts (xy 96.5919 65.278) (xy 97.79 65.278))
     (stroke (width 0) (type default))
   )
@@
     (stroke (width 0) (type default))
   )
-  (wire (pts (xy 95.758 65.278) (xy 97.79 65.278))
+  (wire (pts (xy 95.758 65.278) (xy 96.5919 65.278))
     (stroke (width 0) (type default))
   )
@@
     (stroke (width 0) (type default))
   )
-  (wire (pts (xy 207.518 52.578) (xy 210.058 52.578))
+  (wire (pts (xy 206.248 52.578) (xy 210.058 52.578))
     (stroke (width 0) (type default))
   )
@@
   )
   (rectangle (start 157.226 17.78) (end 282.448 90.932)
-    (stroke (width 0) (type default))
+    (stroke (width 0) (type dash))
     (fill (type none))
   )
-  (rectangle (start 12.7 12.7) (end 156.464 77.724)
+  (rectangle (start 12.7 12.7) (end 156.464 81.28)
     (stroke (width 0) (type dash))
     (fill (type none))
@@
     )
   )
+  (symbol (lib_id "power:GND") (at 96.5919 72.898 0) (unit 1)
+    (in_bom yes) (on_board yes) (dnp no) (fields_autoplaced)
+    (property "Reference" "#PWR030" (at 96.5919 79.248 0)
+      (effects (font (size 1.27 1.27)) hide)
+    )
+    (property "Value" "GND" (at 96.5919 77.978 0)
+      (effects (font (size 1.27 1.27)))
+    )
+    (property "Footprint" "" (at 96.5919 72.898 0)
+      (effects (font (size 1.27 1.27)) hide)
+    )
+    (property "Datasheet" "" (at 96.5919 72.898 0)
+      (effects (font (size 1.27 1.27)) hide)
+    )
+    (pin "1")
+    (instances
+      (project "Drum"
+        (path "/98143dfc-26b3-4fe2-8ea0-3a6505a381c7"
+          (reference "#PWR030") (unit 1)
+        )
+      )
+      (project "VCF"
+        (path "/d6cc6494-bdad-4670-b5b4-2c694da92d9a"
+          (reference "#PWR0113") (unit 1)
+        )
+      )
+    )
+  )
   (symbol (lib_id "Device:R") (at 37.846 110.744 90) (unit 1)
     (in_bom yes) (on_board yes) (dnp no) (fields_autoplaced)
@@
       (effects (font (size 1.27 1.27)) hide)
     )
-    (property "Value" "0R" (at 91.948 69.342 90)
+    (property "Value" "1k" (at 91.948 69.342 90)
       (effects (font (size 1.27 1.27)))
     )
@@
       (effects (font (size 1.27 1.27)) (justify right) hide)
     )
-    (property "Value" "AlpsPot" (at 152.146 40.386 0)
+    (property "Value" "AlpsPot" (at 147.32 55.88 0)
       (effects (font (size 1.27 1.27)))
     )
@@
   )
   (symbol (lib_id "Device:C") (at 99.06 49.53 180) (unit 1)
-    (in_bom yes) (on_board yes) (dnp no) (fields_autoplaced)
+    (in_bom yes) (on_board yes) (dnp no)
     (property "Reference" "C2" (at 102.87 48.26 0)
       (effects (font (size 1.27 1.27)) (justify right) hide)
     )
-    (property "Value" "5n" (at 102.87 50.8 0)
+    (property "Value" "1u to 5u" (at 96.52 43.18 0)
       (effects (font (size 1.27 1.27)) (justify right))
     )
@@
     )
   )
-  (symbol (lib_id "Connector:Conn_01x01_Pin") (at 197.485 40.005 270) (unit 1)
-    (in_bom yes) (on_board yes) (dnp no)
-    (property "Reference" "J4" (at 187.96 33.655 90)
-      (effects (font (size 1.27 1.27)) (justify left) hide)
-    )
-    (property "Value" "Conn_01x11_Pin" (at 187.96 36.195 90)
-      (effects (font (size 1.27 1.27)) (justify left))
-    )
-    (property "Footprint" "Connector_PinHeader_2.54mm:PinHeader_1x01_P2.54mm_Vertical" (at 197.485 40.005 0)
-      (effects (font (size 1.27 1.27)) hide)
-    )
-    (property "Datasheet" "~" (at 197.485 40.005 0)
-      (effects (font (size 1.27 1.27)) hide)
-    )
-    (pin "1")
-    (instances
-      (project "Drum"
-        (path "/98143dfc-26b3-4fe2-8ea0-3a6505a381c7"
-          (reference "J4") (unit 1)
-        )
-      )
-    )
-  )
   (symbol (lib_id "HEJ:AlpsPot") (at 115.316 108.204 0) (unit 1)
     (in_bom yes) (on_board yes) (dnp no)
@@
     )
   )
+  (symbol (lib_id "Device:D") (at 96.5919 69.088 270) (unit 1)
+    (in_bom yes) (on_board yes) (dnp no)
+    (property "Reference" "D4" (at 90.2419 69.088 0)
+      (effects (font (size 1.27 1.27)) hide)
+    )
+    (property "Value" "D" (at 94.0519 71.628 90)
+      (effects (font (size 1.27 1.27)) (justify left))
+    )
+    (property "Footprint" "Diode_THT:D_A-405_P7.62mm_Horizontal" (at 96.5919 69.088 0)
+      (effects (font (size 1.27 1.27)) hide)
+    )
+    (property "Datasheet" "~" (at 96.5919 69.088 0)
+      (effects (font (size 1.27 1.27)) hide)
+    )
+    (property "Sim.Device" "D" (at 96.5919 69.088 0)
+      (effects (font (size 1.27 1.27)) hide)
+    )
+    (property "Sim.Pins" "1=K 2=A" (at 96.5919 69.088 0)
+      (effects (font (size 1.27 1.27)) hide)
+    )
+    (pin "1")
+    (pin "2")
+    (instances
+      (project "Drum"
+        (path "/98143dfc-26b3-4fe2-8ea0-3a6505a381c7"
+          (reference "D4") (unit 1)
+        )
+      )
+    )
+  )
   (symbol (lib_id "power:-12V") (at 118.237 181.102 180) (unit 1)
     (in_bom yes) (on_board yes) (dnp no) (fields_autoplaced)
@@
     )
   )
-  (symbol (lib_id "Device:R") (at 207.518 48.768 180) (unit 1)
-    (in_bom yes) (on_board yes) (dnp no)
-    (property "Reference" "R26" (at 200.914 47.244 0)
-      (effects (font (size 1.27 1.27)) (justify right) hide)
-    )
-    (property "Value" "omit" (at 200.914 49.784 0)
-      (effects (font (size 1.27 1.27)) (justify right))
-    )
-    (property "Footprint" "Resistor_THT:R_Axial_DIN0207_L6.3mm_D2.5mm_P7.62mm_Horizontal" (at 209.296 48.768 90)
-      (effects (font (size 1.27 1.27)) hide)
-    )
-    (property "Datasheet" "~" (at 207.518 48.768 0)
-      (effects (font (size 1.27 1.27)) hide)
-    )
-    (pin "1")
-    (pin "2")
-    (instances
-      (project "Drum"
-        (path "/98143dfc-26b3-4fe2-8ea0-3a6505a381c7"
-          (reference "R26") (unit 1)
-        )
-      )
-      (project "VCF"
-        (path "/d6cc6494-bdad-4670-b5b4-2c694da92d9a"
-          (reference "R11") (unit 1)
-        )
-      )
-    )
-  )
   (symbol (lib_id "power:GND") (at 184.658 72.898 0) (unit 1)
     (in_bom yes) (on_board yes) (dnp no) (fields_autoplaced)
@@
       (effects (font (size 1.27 1.27)) (justify right) hide)
     )
-    (property "Value" "Aux_flush" (at 151.638 45.4152 0)
+    (property "Value" "Aux_flush" (at 152.4 38.1 0)
       (effects (font (size 1.27 1.27)))
     )
@@
   )
   (symbol (lib_id "Device:C") (at 93.98 49.53 180) (unit 1)
-    (in_bom yes) (on_board yes) (dnp no) (fields_autoplaced)
+    (in_bom yes) (on_board yes) (dnp no)
     (property "Reference" "C7" (at 97.79 48.26 0)
       (effects (font (size 1.27 1.27)) (justify right) hide)
     )
-    (property "Value" "5n" (at 97.79 50.8 0)
-      (effects (font (size 1.27 1.27)) (justify right))
+    (property "Value" "5n" (at 96.52 53.34 0)
+      (effects (font (size 1.27 1.27)) (justify right) hide)
     )
     (property "Footprint" "Capacitor_THT:C_Axial_L5.1mm_D3.1mm_P7.50mm_Horizontal" (at 93.0148 45.72 0)
@@
       (effects (font (size 1.27 1.27)) (justify right) hide)
     )
-    (property "Value" "1k" (at 145.288 38.1 90)
+    (property "Value" "100k" (at 145.288 38.1 90)
       (effects (font (size 1.27 1.27)))
     )
@@
       (effects (font (size 1.27 1.27)) (justify left) hide)
     )
-    (property "Value" "BC557" (at 96.012 71.374 0)
+    (property "Value" "BC557" (at 104.14 73.66 0)
       (effects (font (size 1.27 1.27)) (justify left))
     )
