File: Hat/Hat.kicad_sch (KiCad schematic)
At the start: 86 parts, among them J1 Conn_01x01_Pin, J2 Conn_01x12_Pin, J3 Conn_01x12_Pin, J4 Conn_01x06_Pin, Q1 BC547, Q10 BC547, Q3 BC547, Q4 BC547, Q6 BC547, Q7 BC547, Q8 BC547, Q8 BC557, SW1 SW_Push, SW2 SW_SPDT, U1 TL074, U13 Aux_flush, U5 4066

Commit message: Add files via upload
Parts:
- C3: value 470n -> 220n
Changed lines of the file:
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@@
       (effects (font (size 1.27 1.27)) hide)
     )
-    (property "Value" "470n" (at 66.294 95.25 90)
+    (property "Value" "220n" (at 66.294 95.25 90)
       (effects (font (size 1.27 1.27)))
     )
