File: MIDI-Interface/MIDI-BackBoard2/MIDI-BackBoard2.kicad_pcb (KiCad board)
At the start: 2 copper layers, 43.8 x 93.3 mm, 35 parts, among them J1 Conn_01x06_Pin, J5 Conn_01x14_Pin, U1 TL074, U2 L7806, U3 EL817, U4 TL072, U5 TL074

Commit message: Add files via upload
Parts:
- added J2: Conn_01x01_Pin, Connector_PinHeader_2.54mm:PinHeader_1x01_P2.54mm_Vertical, F.Cu at (147.8, 135.1)
Connections:
- A1 pad 20: unconnected-(A1-A1-Pad20) -> D4
- A1 pad 21: unconnected-(A1-A2-Pad21) -> D3
- A1 pad 25: D4 -> unconnected-(A1-A6-Pad25)
- A1 pad 26: D3 -> unconnected-(A1-A7-Pad26)
Routing:
- net D3: track 37.4 -> 50.1 mm
- net D4: track 46.4 -> 57.3 mm
- net MIDI_DATA: track 62.5 -> 71.7 mm
Changed lines of the file:
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@@
   (net 9 "ENCB")
   (net 10 "D1")
-  (net 11 "unconnected-(A1-A1-Pad20)")
-  (net 12 "unconnected-(A1-A2-Pad21)")
+  (net 11 "unconnected-(A1-A6-Pad25)")
+  (net 12 "unconnected-(A1-A7-Pad26)")
   (net 13 "SW")
   (net 14 "unconnected-(A1-A3-Pad22)")
@@
       (net 19 "unconnected-(A1-A0-Pad19)") (pinfunction "A0") (pintype "bidirectional"))
     (pad "20" thru_hole oval (at 15.24 25.4) (size 1.6 1.6) (drill 1) (layers "*.Cu" "*.Mask")
-      (net 11 "unconnected-(A1-A1-Pad20)") (pinfunction "A1") (pintype "bidirectional"))
+      (net 7 "D4") (pinfunction "A1") (pintype "bidirectional"))
     (pad "21" thru_hole oval (at 15.24 22.86) (size 1.6 1.6) (drill 1) (layers "*.Cu" "*.Mask")
-      (net 12 "unconnected-(A1-A2-Pad21)") (pinfunction "A2") (pintype "bidirectional"))
+      (net 6 "D3") (pinfunction "A2") (pintype "bidirectional"))
     (pad "22" thru_hole oval (at 15.24 20.32) (size 1.6 1.6) (drill 1) (layers "*.Cu" "*.Mask")
       (net 14 "unconnected-(A1-A3-Pad22)") (pinfunction "A3") (pintype "bidirectional"))
@@
       (net 24 "unconnected-(A1-SCL{slash}A5-Pad24)") (pinfunction "SCL/A5") (pintype "bidirectional"))
     (pad "25" thru_hole oval (at 15.24 12.7) (size 1.6 1.6) (drill 1) (layers "*.Cu" "*.Mask")
-      (net 7 "D4") (pinfunction "A6") (pintype "bidirectional"))
+      (net 11 "unconnected-(A1-A6-Pad25)") (pinfunction "A6") (pintype "bidirectional"))
     (pad "26" thru_hole oval (at 15.24 10.16) (size 1.6 1.6) (drill 1) (layers "*.Cu" "*.Mask")
-      (net 6 "D3") (pinfunction "A7") (pintype "bidirectional"))
+      (net 12 "unconnected-(A1-A7-Pad26)") (pinfunction "A7") (pintype "bidirectional"))
     (pad "27" thru_hole oval (at 15.24 7.62) (size 1.6 1.6) (drill 1) (layers "*.Cu" "*.Mask")
       (net 25 "+5V") (pinfunction "+5V") (pintype "power_out"))
@@
     )
   )
+  (footprint "Connector_PinHeader_2.54mm:PinHeader_1x01_P2.54mm_Vertical" (layer "F.Cu")
+    (at 147.8 135.1)
+    (descr "Through hole straight pin header, 1x01, 2.54mm pitch, single row")
+    (tags "Through hole pin header THT 1x01 2.54mm single row")
+    (property "Sheetfile" "MIDI-BackBoard2.kicad_sch")
+    (property "Sheetname" "")
+    (property "ki_description" "Generic connector, single row, 01x01, script generated")
+    (property "ki_keywords" "connector")
+    (attr through_hole)
+    (fp_text reference "J2" (at 0 -2.33) (layer "F.SilkS") hide
+        (effects (font (size 1 1) (thickness 0.15)))
+    )
+    (fp_text value "Conn_01x01_Pin" (at 0 2.33) (layer "F.Fab")
+        (effects (font (size 1 1) (thickness 0.15)))
+    )
+    (fp_text user "${REFERENCE}" (at 0 0 90) (layer "F.Fab")
+        (effects (font (size 1 1) (thickness 0.15)))
+    )
+    (fp_line (start -1.33 -1.33) (end 0 -1.33)
+      (stroke (width 0.12) (type solid)) (layer "F.SilkS"))
+    (fp_line (start -1.33 0) (end -1.33 -1.33)
+      (stroke (width 0.12) (type solid)) (layer "F.SilkS"))
+    (fp_line (start -1.33 1.27) (end -1.33 1.33)
+      (stroke (width 0.12) (type solid)) (layer "F.SilkS"))
+    (fp_line (start -1.33 1.27) (end 1.33 1.27)
+      (stroke (width 0.12) (type solid)) (layer "F.SilkS"))
+    (fp_line (start -1.33 1.33) (end 1.33 1.33)
+      (stroke (width 0.12) (type solid)) (layer "F.SilkS"))
+    (fp_line (start 1.33 1.27) (end 1.33 1.33)
+      (stroke (width 0.12) (type solid)) (layer "F.SilkS"))
+    (fp_line (start -1.8 -1.8) (end -1.8 1.8)
+      (stroke (width 0.05) (type solid)) (layer "F.CrtYd"))
+    (fp_line (start -1.8 1.8) (end 1.8 1.8)
+      (stroke (width 0.05) (type solid)) (layer "F.CrtYd"))
+    (fp_line (start 1.8 -1.8) (end -1.8 -1.8)
+      (stroke (width 0.05) (type solid)) (layer "F.CrtYd"))
+    (fp_line (start 1.8 1.8) (end 1.8 -1.8)
+      (stroke (width 0.05) (type solid)) (layer "F.CrtYd"))
+    (fp_line (start -1.27 -0.635) (end -0.635 -1.27)
+      (stroke (width 0.1) (type solid)) (layer "F.Fab"))
+    (fp_line (start -1.27 1.27) (end -1.27 -0.635)
+      (stroke (width 0.1) (type solid)) (layer "F.Fab"))
+    (fp_line (start -0.635 -1.27) (end 1.27 -1.27)
+      (stroke (width 0.1) (type solid)) (layer "F.Fab"))
+    (fp_line (start 1.27 -1.27) (end 1.27 1.27)
+      (stroke (width 0.1) (type solid)) (layer "F.Fab"))
+    (fp_line (start 1.27 1.27) (end -1.27 1.27)
+      (stroke (width 0.1) (type solid)) (layer "F.Fab"))
+    (pad "1" thru_hole rect (at 0 0) (size 1.7 1.7) (drill 1) (layers "*.Cu" "*.Mask")
+      (net 2 "MIDI_DATA") (pinfunction "Pin_1") (pintype "passive"))
+    (model "${KICAD6_3DMODEL_DIR}/Connector_PinHeader_2.54mm.3dshapes/PinHeader_1x01_P2.54mm_Vertical.wrl"
+      (offset (xyz 0 0 0))
+      (scale (xyz 1 1 1))
+      (rotate (xyz 0 0 0))
+    )
+  )
   (footprint "Resistor_THT:R_Axial_DIN0207_L6.3mm_D2.5mm_P7.62mm_Horizontal" (layer "F.Cu")
     (at 175.27 68.09)
@@
   (gr_line (start 187.78 137.79) (end 144 137.79)
     (stroke (width 0.1) (type default)) (layer "Edge.Cuts"))
+  (segment (start 149.7 135.1) (end 153.14 131.66) (width 0.4) (layer "B.Cu") (net 2))
   (segment (start 155.53 131.66) (end 155.53 133.74) (width 0.4) (layer "B.Cu") (net 2))
   (segment (start 169.52 136.15) (end 174.03 131.64) (width 0.4) (layer "B.Cu") (net 2))
+  (segment (start 153.14 131.66) (end 155.53 131.66) (width 0.4) (layer "B.Cu") (net 2))
   (segment (start 155.53 129.12) (end 155.53 131.66) (width 0.4) (layer "B.Cu") (net 2))
   (segment (start 155.53 133.74) (end 157.94 136.15) (width 0.4) (layer "B.Cu") (net 2))
@@
   (segment (start 157.94 136.15) (end 169.52 136.15) (width 0.4) (layer "B.Cu") (net 2))
   (segment (start 174.03 131.64) (end 174.03 106.84) (width 0.4) (layer "B.Cu") (net 2))
+  (segment (start 147.8 135.1) (end 149.7 135.1) (width 0.4) (layer "B.Cu") (net 2))
   (segment (start 174.03 106.84) (end 166.92 99.73) (width 0.4) (layer "B.Cu") (net 2))
   (segment (start 156.68 103.62) (end 156.68 102.19) (width 0.4) (layer "F.Cu") (net 4))
@@
   (segment (start 166.62 107.35) (end 167.18 106.79) (width 0.4) (layer "F.Cu") (net 5))
   (segment (start 165.22 107.35) (end 166.62 107.35) (width 0.4) (layer "F.Cu") (net 5))
-  (segment (start 184.38 85.29) (end 184.38 103.43) (width 0.4) (layer "F.Cu") (net 6))
+  (segment (start 173.68 84.49) (end 183.58 84.49) (width 0.4) (layer "F.Cu") (net 6))
+  (segment (start 172.695 85.475) (end 173.68 84.49) (width 0.4) (layer "F.Cu") (net 6))
+  (segment (start 183.58 84.49) (end 184.38 85.29) (width 0.4) (layer "F.Cu") (net 6))
+  (segment (start 184.38 116.13) (end 180.46 120.05) (width 0.4) (layer "F.Cu") (net 6))
   (segment (start 171.45 85.475) (end 172.695 85.475) (width 0.4) (layer "F.Cu") (net 6))
-  (segment (start 172.695 85.475) (end 173.68 84.49) (width 0.4) (layer "F.Cu") (net 6))
-  (segment (start 173.68 84.49) (end 183.58 84.49) (width 0.4) (layer "F.Cu") (net 6))
-  (segment (start 184.38 103.43) (end 180.46 107.35) (width 0.4) (layer "F.Cu") (net 6))
-  (segment (start 183.58 84.49) (end 184.38 85.29) (width 0.4) (layer "F.Cu") (net 6))
+  (segment (start 184.38 85.29) (end 184.38 116.13) (width 0.4) (layer "F.Cu") (net 6))
   (segment (start 171.45 80.395) (end 172.085 80.395) (width 0.4) (layer "F.Cu") (net 7))
   (segment (start 173.78 82.09) (end 185.5 82.09) (width 0.4) (layer "F.Cu") (net 7))
-  (segment (start 183.48 109.89) (end 180.46 109.89) (width 0.4) (layer "F.Cu") (net 7))
-  (segment (start 185.5 82.09) (end 185.5 107.87) (width 0.4) (layer "F.Cu") (net 7))
   (segment (start 172.085 80.395) (end 173.78 82.09) (width 0.4) (layer "F.Cu") (net 7))
-  (segment (start 185.5 107.87) (end 183.48 109.89) (width 0.4) (layer "F.Cu") (net 7))
+  (segment (start 185.5 117.55) (end 180.46 122.59) (width 0.4) (layer "F.Cu") (net 7))
+  (segment (start 185.5 82.09) (end 185.5 117.55) (width 0.4) (layer "F.Cu") (net 7))
   (segment (start 151.18 99.99) (end 151.18 98.89) (width 0.4) (layer "B.Cu") (net 8))
   (segment (start 155.28 104.09) (end 151.18 99.99) (width 0.4) (layer "B.Cu") (net 8))
