File: MIDI-Interface/MIDI-BackBoard2/MIDI-BackBoard2.kicad_sch (KiCad schematic)
At the start: 35 parts, among them J1 Conn_01x06_Pin, J5 Conn_01x14_Pin, U1 TL074, U2 L7806, U3 EL817, U4 TL072, U5 TL074

Commit message: Add files via upload
Parts:
- added J2: Conn_01x01_Pin, Connector_PinHeader_2.54mm:PinHeader_1x01_P2.54mm_Vertical, symbol Connector:Conn_01x01_Pin
Connections:
- net D3: now also A1.21 (A2); no longer A1.26 (A7)
- net D4: now also A1.20 (A1); no longer A1.25 (A6)
- net MIDI_DATA: now also J2.1 (Pin_1)
Changed lines of the file:
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@@
   (junction (at 210.82 134.62) (diameter 0) (color 0 0 0 0)
   )
+  (junction (at 93.98 45.72) (diameter 0) (color 0 0 0 0)
+  )
   (junction (at 254 134.62) (diameter 0) (color 0 0 0 0)
   )
@@
   )
   (wire (pts (xy 147.32 167.64) (xy 162.56 167.64))
+    (stroke (width 0) (type default))
+  )
+  (wire (pts (xy 93.98 45.72) (xy 101.6 45.72))
     (stroke (width 0) (type default))
   )
@@
     )
   )
-  (global_label "D4" (shape input) (at 73.66 111.76 0) (fields_autoplaced)
-    (effects (font (size 1.27 1.27)) (justify left))
-    (property "Intersheetrefs" "${INTERSHEET_REFS}" (at 79.1247 111.76 0)
+  (global_label "D4" (shape input) (at 73.66 99.06 0) (fields_autoplaced)
+    (effects (font (size 1.27 1.27)) (justify left))
+    (property "Intersheetrefs" "${INTERSHEET_REFS}" (at 79.1247 99.06 0)
       (effects (font (size 1.27 1.27)) (justify left) hide)
     )
@@
     )
   )
-  (global_label "D3" (shape input) (at 73.66 114.3 0) (fields_autoplaced)
-    (effects (font (size 1.27 1.27)) (justify left))
-    (property "Intersheetrefs" "${INTERSHEET_REFS}" (at 79.1247 114.3 0)
+  (global_label "D3" (shape input) (at 73.66 101.6 0) (fields_autoplaced)
+    (effects (font (size 1.27 1.27)) (justify left))
+    (property "Intersheetrefs" "${INTERSHEET_REFS}" (at 79.1247 101.6 0)
       (effects (font (size 1.27 1.27)) (justify left) hide)
     )
@@
         )
       )
+    )
+  )
+  (symbol (lib_id "Connector:Conn_01x01_Pin") (at 106.68 45.72 180) (unit 1)
+    (in_bom yes) (on_board yes) (dnp no)
+    (property "Reference" "J2" (at 106.68 48.26 0)
+      (effects (font (size 1.27 1.27)))
+    )
+    (property "Value" "Conn_01x01_Pin" (at 106.68 50.8 0)
+      (effects (font (size 1.27 1.27)))
+    )
+    (property "Footprint" "Connector_PinHeader_2.54mm:PinHeader_1x01_P2.54mm_Vertical" (at 106.68 45.72 0)
+      (effects (font (size 1.27 1.27)) hide)
+    )
+    (property "Datasheet" "~" (at 106.68 45.72 0)
+      (effects (font (size 1.27 1.27)) hide)
+    )
+    (pin "1")
+    (instances
+      (project "MIDI-BackBoard2"
+        (path "/6533e9e1-cddb-41b9-b1bd-8b2ec03ab641"
+          (reference "J2") (unit 1)
+        )
+      )
