File: Euclid/Euclid.kicad_pcb (KiCad board)
At the start: 2 copper layers, 129.5 x 128.5 mm, 73 parts, among them J1 Conn_01x06_Pin, J10 Conn_01x01_Pin, J11 Conn_01x01_Pin, J12 Conn_01x01_Pin, J13 Conn_01x01_Pin, J14 Conn_01x01_Pin, J15 Conn_01x01_Pin, J16 Conn_01x01_Pin, J17 Conn_01x01_Pin, J2 Conn_01x12_Pin, J3 Conn_01x12_Pin, J4 Conn_01x01_Pin, J5 Conn_01x01_Pin, J6 Conn_01x01_Pin, J7 Conn_01x01_Pin, J8 Conn_01x01_Pin, J9 Conn_01x01_Pin, Q1 BC547, Q3 BC547, U1 Aux_flush, U4 L7805, U5 Aux_flush, U6 Aux_flush, U7 TL072, U8 Aux_flush, U9 Aux_flush

Commit message: Add files via upload
Connections:
- R13 pad 1: +12V -> +5V
- R7 pad 1: +12V -> +5V
Routing:
- net +5V: track 63.3 -> 114.1 mm
Changed lines of the file:
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@@
       (stroke (width 0.1) (type solid)) (layer "F.Fab"))
     (pad "1" thru_hole circle (at 0 0 180) (size 1.6 1.6) (drill 0.8) (layers "*.Cu" "*.Mask")
-      (net 19 "+12V") (pintype "passive"))
+      (net 21 "+5V") (pintype "passive"))
     (pad "2" thru_hole oval (at 7.62 0 180) (size 1.6 1.6) (drill 0.8) (layers "*.Cu" "*.Mask")
       (net 45 "RESET_BUTTON") (pintype "passive"))
@@
       (stroke (width 0.1) (type solid)) (layer "F.Fab"))
     (pad "1" thru_hole circle (at 0 0 180) (size 1.6 1.6) (drill 0.8) (layers "*.Cu" "*.Mask")
-      (net 19 "+12V") (pintype "passive"))
+      (net 21 "+5V") (pintype "passive"))
     (pad "2" thru_hole oval (at 7.62 0 180) (size 1.6 1.6) (drill 0.8) (layers "*.Cu" "*.Mask")
       (net 44 "SHFT_BUTTON") (pintype "passive"))
@@
     (property "Sheetname" "")
     (attr through_hole)
-    (fp_text reference "U5" (at 2.1 -7.45 90) (layer "F.SilkS")
+    (fp_text reference "U5" (at 2.1 -7.45 90) (layer "F.SilkS") hide
         (effects (font (size 1 1) (thickness 0.15)))
     )
@@
     (property "Sheetname" "")
     (attr through_hole)
-    (fp_text reference "U1" (at 2.1 -7.45 90) (layer "F.SilkS")
+    (fp_text reference "U1" (at 2.1 -7.45 90) (layer "F.SilkS") hide
         (effects (font (size 1 1) (thickness 0.15)))
     )
@@
   (segment (start 207.93 80.83) (end 211.01 80.83) (width 0.4) (layer "F.Cu") (net 20))
   (segment (start 203.39 78.29) (end 205.39 78.29) (width 0.4) (layer "F.Cu") (net 20))
-  (segment (start 209.083528 115.153528) (end 208.727057 115.51) (width 0.4) (layer "F.Cu") (net 21))
-  (segment (start 213.19 119.26) (end 213 119.07) (width 0.4) (layer "F.Cu") (net 21))
-  (segment (start 200.18 89.57) (end 205.23 89.57) (width 0.4) (layer "F.Cu") (net 21))
-  (segment (start 198 104.07) (end 198 91.75) (width 0.4) (layer "F.Cu") (net 21))
-  (segment (start 208.727057 115.51) (end 207.732943 115.51) (width 0.4) (layer "F.Cu") (net 21))
-  (segment (start 216.67 119.07) (end 213 119.07) (width 0.4) (layer "F.Cu") (net 21))
-  (segment (start 198 91.75) (end 200.18 89.57) (width 0.4) (layer "F.Cu") (net 21))
+  (segment (start 216.67 119.07) (end 198.68 119.07) (width 0.4) (layer "F.Cu") (net 21))
+  (segment (start 200.18 89.57) (end 198 91.75) (width 0.4) (layer "F.Cu") (net 21))
+  (segment (start 198 105.15) (end 223.85 105.15) (width 0.4) (layer "F.Cu") (net 21))
+  (segment (start 205.23 89.57) (end 200.18 89.57) (width 0.4) (layer "F.Cu") (net 21))
+  (segment (start 223.85 105.15) (end 226.5 102.5) (width 0.4) (layer "F.Cu") (net 21))
+  (segment (start 205.23 89.57) (end 205.23 91.03) (width 0.4) (layer "F.Cu") (net 21))
+  (segment (start 207.35 93.15) (end 213.2 93.15) (width 0.4) (layer "F.Cu") (net 21))
+  (segment (start 205.23 91.03) (end 207.35 93.15) (width 0.4) (layer "F.Cu") (net 21))
+  (segment (start 198 118.39) (end 198.68 119.07) (width 0.4) (layer "F.Cu") (net 21))
   (segment (start 213.19 121.79) (end 213.19 119.26) (width 0.4) (layer "F.Cu") (net 21))
-  (segment (start 207.03 114.807057) (end 207.03 113.1) (width 0.4) (layer "F.Cu") (net 21))
-  (segment (start 213 119.07) (end 209.083528 115.153528) (width 0.4) (layer "F.Cu") (net 21))
-  (segment (start 207.732943 115.51) (end 207.03 114.807057) (width 0.4) (layer "F.Cu") (net 21))
-  (segment (start 207.03 113.1) (end 198 104.07) (width 0.4) (layer "F.Cu") (net 21))
+  (segment (start 198 105.15) (end 198 118.39) (width 0.4) (layer "F.Cu") (net 21))
+  (segment (start 216.31 95.5) (end 213.96 93.15) (width 0.4) (layer "F.Cu") (net 21))
+  (segment (start 213.96 93.15) (end 213.2 93.15) (width 0.4) (layer "F.Cu") (net 21))
+  (segment (start 198 91.75) (end 198 105.15) (width 0.4) (layer "F.Cu") (net 21))
   (segment (start 226.11 116.75) (end 228.55 114.31) (width 0.4) (layer "B.Cu") (net 21))
   (segment (start 216.67 119.07) (end 218.99 116.75) (width 0.4) (layer "B.Cu") (net 21))
@@
     )
   )
-  (group "" (id 3d0918ad-58ab-4c1d-8e32-dba996e40daa)
+  (group "" (id f2cb1453-1de8-47b6-94ad-2057980465de)
     (members
       0e3a9408-cb3a-4ee0-a33c-ff872b00eaa6
