File: Euclid/Euclid.kicad_sch (KiCad schematic)
At the start: 56 parts, among them J1 Conn_01x06_Pin, J10 Conn_01x01_Pin, J11 Conn_01x01_Pin, J12 Conn_01x01_Pin, J13 Conn_01x01_Pin, J14 Conn_01x01_Pin, J15 Conn_01x01_Pin, J16 Conn_01x01_Pin, J17 Conn_01x01_Pin, J2 Conn_01x12_Pin, J3 Conn_01x12_Pin, J4 Conn_01x01_Pin, J5 Conn_01x01_Pin, J6 Conn_01x01_Pin, J7 Conn_01x01_Pin, J8 Conn_01x01_Pin, J9 Conn_01x01_Pin, Q1 BC547, Q3 BC547, SW1 SW_Push, SW2 SW_Push, U1 Aux_flush, U4 L7805, U5 Aux_flush, U6 Aux_flush, U7 TL072, U8 Aux_flush, U9 Aux_flush

Commit message: Add files via upload
Connections:
- net +12V: no longer R13.1, R7.1
- net +5V: now also R13.1, R7.1
Changed lines of the file:
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@@
     )
   )
-  (symbol (lib_id "power:+12V") (at 81.28 123.19 0) (unit 1)
-    (in_bom yes) (on_board yes) (dnp no) (fields_autoplaced)
-    (property "Reference" "#PWR036" (at 81.28 127 0)
-      (effects (font (size 1.27 1.27)) hide)
-    )
-    (property "Value" "+12V" (at 81.28 118.11 0)
+  (symbol (lib_id "power:+5V") (at 81.28 123.19 0) (unit 1)
+    (in_bom yes) (on_board yes) (dnp no) (fields_autoplaced)
+    (property "Reference" "#PWR034" (at 81.28 127 0)
+      (effects (font (size 1.27 1.27)) hide)
+    )
+    (property "Value" "+5V" (at 81.28 118.11 0)
       (effects (font (size 1.27 1.27)))
     )
@@
       (project "Euclid"
         (path "/9cc2e01f-5694-4849-bf93-19792a9718f5"
-          (reference "#PWR036") (unit 1)
+          (reference "#PWR034") (unit 1)
         )
       )
@@
     )
   )
+  (symbol (lib_id "power:+5V") (at 114.3 123.19 0) (unit 1)
+    (in_bom yes) (on_board yes) (dnp no) (fields_autoplaced)
+    (property "Reference" "#PWR036" (at 114.3 127 0)
+      (effects (font (size 1.27 1.27)) hide)
+    )
+    (property "Value" "+5V" (at 114.3 118.11 0)
+      (effects (font (size 1.27 1.27)))
+    )
+    (property "Footprint" "" (at 114.3 123.19 0)
+      (effects (font (size 1.27 1.27)) hide)
+    )
+    (property "Datasheet" "" (at 114.3 123.19 0)
+      (effects (font (size 1.27 1.27)) hide)
+    )
+    (pin "1")
+    (instances
+      (project "Euclid"
+        (path "/9cc2e01f-5694-4849-bf93-19792a9718f5"
+          (reference "#PWR036") (unit 1)
+        )
+      )
+    )
+  )
   (symbol (lib_id "Device:D") (at 58.42 76.2 270) (unit 1)
     (in_bom yes) (on_board yes) (dnp no) (fields_autoplaced)
@@
         )
       )
-    )
-  )
-  (symbol (lib_id "power:+12V") (at 114.3 123.19 0) (unit 1)
-    (in_bom yes) (on_board yes) (dnp no) (fields_autoplaced)
-    (property "Reference" "#PWR034" (at 114.3 127 0)
-      (effects (font (size 1.27 1.27)) hide)
-    )
-    (property "Value" "+12V" (at 114.3 118.11 0)
-      (effects (font (size 1.27 1.27)))
-    )
-    (property "Footprint" "" (at 114.3 123.19 0)
-      (effects (font (size 1.27 1.27)) hide)
-    )
-    (property "Datasheet" "" (at 114.3 123.19 0)
-      (effects (font (size 1.27 1.27)) hide)
-    )
-    (pin "1")
-    (instances
-      (project "Euclid"
-        (path "/9cc2e01f-5694-4849-bf93-19792a9718f5"
-          (reference "#PWR034") (unit 1)
-        )
-      )
