File: 3360_CrossFader/3360_CrossFader.kicad_pcb (KiCad board)
At the start: 2 copper layers, 110 x 128 mm, 60 parts, among them J1 Conn_01x06_Male, J2 Conn_01x06_Male, J3 Conn_01x08_Pin, J5 Conn_01x08_Pin, J6 Conn_01x06_Male, Q1 BC547, Q2 BC547, U1 Aux_flush, U10 Aux_flush, U11 Aux_flush, U2 TL074, U3 TL072, U4 Aux_flush, U5 Aux_flush, U6 AS3360, U7 Switch, U8 Aux_flush, U9 Aux_flush

Commit message: Add files via upload
Updated PCB
Routing:
- net GND: track 0.00 -> 10.1 mm
Changed lines of the file:
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@@
   (segment (start 157.417463 102.395885) (end 165.167463 102.395885) (width 0.4) (layer "F.Cu") (net 1))
   (segment (start 156.802463 103.010885) (end 157.417463 102.395885) (width 0.4) (layer "F.Cu") (net 1))
+  (segment (start 144.3 73.45) (end 144.3 69.45) (width 0.4) (layer "F.Cu") (net 2))
+  (segment (start 144.780885 73.930885) (end 144.3 73.45) (width 0.4) (layer "F.Cu") (net 2))
+  (segment (start 144.899115 68.850885) (end 147.117463 68.850885) (width 0.4) (layer "F.Cu") (net 2))
+  (segment (start 144.3 69.45) (end 144.899115 68.850885) (width 0.4) (layer "F.Cu") (net 2))
+  (segment (start 147.117463 73.930885) (end 144.780885 73.930885) (width 0.4) (layer "F.Cu") (net 2))
   (segment (start 133.917463 97.205885) (end 136.647463 97.205885) (width 0.4) (layer "F.Cu") (net 3))
   (segment (start 136.647463 97.205885) (end 136.917463 97.475885) (width 0.4) (layer "F.Cu") (net 3))
@@
   (segment (start 224.497463 101.395885) (end 219.997463 101.395885) (width 0.4) (layer "B.Cu") (net 40))
   (segment (start 195.567113 122.465535) (end 187.997463 122.465535) (width 0.4) (layer "B.Cu") (net 40))
+  (segment (start 175.9 106.413348) (end 174.727463 107.585885) (width 0.4) (layer "B.Cu") (net 40))
   (segment (start 227.997463 107.585885) (end 225.687463 107.585885) (width 0.4) (layer "B.Cu") (net 40))
-  (segment (start 168.997463 78.395885) (end 174.917463 78.395885) (width 0.4) (layer "B.Cu") (net 40))
   (segment (start 214.997463 134.895885) (end 197.997463 134.895885) (width 0.4) (layer "B.Cu") (net 40))
   (segment (start 219.997463 101.395885) (end 214.997463 106.395885) (width 0.4) (layer "B.Cu") (net 40))
   (segment (start 224.497463 106.395885) (end 224.497463 101.395885) (width 0.4) (layer "B.Cu") (net 40))
-  (segment (start 175.417463 106.895885) (end 174.727463 107.585885) (width 0.4) (layer "B.Cu") (net 40))
+  (segment (start 174.917463 78.395885) (end 175.9 79.378422) (width 0.4) (layer "B.Cu") (net 40))
   (segment (start 225.687463 107.585885) (end 224.497463 106.395885) (width 0.4) (layer "B.Cu") (net 40))
-  (segment (start 174.917463 78.395885) (end 175.417463 78.895885) (width 0.4) (layer "B.Cu") (net 40))
   (segment (start 197.997463 134.895885) (end 195.997463 132.895885) (width 0.4) (layer "B.Cu") (net 40))
-  (segment (start 175.417463 78.895885) (end 175.417463 106.895885) (width 0.4) (layer "B.Cu") (net 40))
   (segment (start 174.727463 107.585885) (end 173.917463 107.585885) (width 0.4) (layer "B.Cu") (net 40))
+  (segment (start 175.9 79.378422) (end 175.9 106.413348) (width 0.4) (layer "B.Cu") (net 40))
+  (segment (start 168.997463 78.395885) (end 174.917463 78.395885) (width 0.4) (layer "B.Cu") (net 40))
   (segment (start 214.997463 106.395885) (end 214.997463 134.895885) (width 0.4) (layer "B.Cu") (net 40))
   (segment (start 195.997463 132.895885) (end 195.997463 122.895885) (width 0.4) (layer "B.Cu") (net 40))
