File: CV_Trigger_Sequencer/DrumSequencer/DrumSequencer.kicad_pcb (KiCad board)
At the start: 2 copper layers, 200.3 x 128 mm, 177 parts, among them J1 Conn_01x06_Male, J2 Conn_01x06_Male, Q1 NDT3055L, Q19 BC547, Q20 BC547, Q21 BC547, Q22 BC547, Q23 BC547, Q24 BC547, Q25 BC547, Q26 BC547, Q27 BC547, Q28 BC547, Q3 BC547, Q4 BC557, Q8 BC547, SW2 SW_Push, U1 TL074, U10 Switch, U11 Switch, U12 Switch, U13 Switch, U14 Switch, U15 Switch, U16 SP3T, U17 SP3T, U18 SP3T, U19 SP3T, U2 TL072, U20 SP3T, U21 SP3T, U22 SP3T, U23 SP3T, U24 Aux_flush, U25 Aux_flush, U26 Aux_flush, U3 TL074, U30 Aux_flush, U31 Aux_flush, U32 Aux_flush, U33 Aux_flush, U34 LM7805_TO220, U35 ATmega328-P, U4 Aux_flush, U6 Aux_flush, U7 Aux_flush, U8 Switch, U9 Switch, Y1 Crystal

Commit message: Add files via upload
Connections:
- U35 pad 1: IN1 -> unconnected-(U35-~{RESET}/PC6-Pad1)
- U35 pad 25: unconnected-(U35-PC2-Pad25) -> IN1
Routing:
- net IN1: track 12.6 -> 33.2 mm
- net Net-(D37-A): track 29.0 -> 29.7 mm
Changed lines of the file:
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@@
   (net 145 "unconnected-(U35-PB5-Pad19)")
   (net 146 "unconnected-(U35-PC5-Pad28)")
-  (net 147 "unconnected-(U35-PC2-Pad25)")
+  (net 147 "unconnected-(U35-~{RESET}{slash}PC6-Pad1)")
   (net 148 "unconnected-(U35-PC4-Pad27)")
   (net 149 "THR")
@@
       (stroke (width 0.1) (type solid)) (layer "F.Fab"))
     (pad "1" thru_hole rect (at 0 0 90) (size 1.6 1.6) (drill 0.8) (layers "*.Cu" "*.Mask")
-      (net 132 "IN1") (pinfunction "~{RESET}/PC6") (pintype "bidirectional"))
+      (net 147 "unconnected-(U35-~{RESET}{slash}PC6-Pad1)") (pinfunction "~{RESET}/PC6") (pintype "bidirectional"))
     (pad "2" thru_hole oval (at 0 2.54 90) (size 1.6 1.6) (drill 0.8) (layers "*.Cu" "*.Mask")
       (net 135 "Net-(U35-PD0)") (pinfunction "PD0") (pintype "bidirectional"))
@@
       (net 76 "A6") (pinfunction "PC1") (pintype "bidirectional"))
     (pad "25" thru_hole oval (at 7.62 7.62 90) (size 1.6 1.6) (drill 0.8) (layers "*.Cu" "*.Mask")
-      (net 147 "unconnected-(U35-PC2-Pad25)") (pinfunction "PC2") (pintype "bidirectional"))
+      (net 132 "IN1") (pinfunction "PC2") (pintype "bidirectional"))
     (pad "26" thru_hole oval (at 7.62 5.08 90) (size 1.6 1.6) (drill 0.8) (layers "*.Cu" "*.Mask")
       (net 128 "Net-(U35-PC3)") (pinfunction "PC3") (pintype "bidirectional"))
@@
   (segment (start 219.152 128.834) (end 222.767 128.834) (width 0.4) (layer "B.Cu") (net 52))
   (segment (start 222.767 128.834) (end 223.887 127.714) (width 0.4) (layer "B.Cu") (net 52))
-  (segment (start 115.212 123.964) (end 119.302 123.964) (width 0.4) (layer "F.Cu") (net 53))
-  (segment (start 119.302 123.964) (end 119.402 124.064) (width 0.4) (layer "F.Cu") (net 53))
   (segment (start 126.902 133.464) (end 137.789966 133.464) (width 0.4) (layer "F.Cu") (net 53))
-  (segment (start 119.402 125.964) (end 126.902 133.464) (width 0.4) (layer "F.Cu") (net 53))
+  (segment (start 115.962 123.214) (end 118.552 123.214) (width 0.4) (layer "F.Cu") (net 53))
+  (segment (start 120.702 127.264) (end 126.902 133.464) (width 0.4) (layer "F.Cu") (net 53))
   (segment (start 137.789966 133.464) (end 138.789966 132.464) (width 0.4) (layer "F.Cu") (net 53))
-  (segment (start 119.402 124.064) (end 119.402 125.964) (width 0.4) (layer "F.Cu") (net 53))
+  (segment (start 115.212 123.964) (end 115.962 123.214) (width 0.4) (layer "F.Cu") (net 53))
+  (segment (start 120.702 125.364) (end 120.702 127.264) (width 0.4) (layer "F.Cu") (net 53))
+  (segment (start 118.552 123.214) (end 120.702 125.364) (width 0.4) (layer "F.Cu") (net 53))
   (segment (start 93.902 112.642) (end 90.63 109.37) (width 0.4) (layer "F.Cu") (net 54))
   (segment (start 95.802 128.384) (end 93.902 126.484) (width 0.4) (layer "F.Cu") (net 54))
@@
   (segment (start 101.512 104.964) (end 103.212 106.664) (width 0.4) (layer "B.Cu") (net 131))
   (segment (start 151.602 108.264) (end 151.602 128.464) (width 0.4) (layer "B.Cu") (net 131))
-  (segment (start 109.202 119.864) (end 109.202 120.954) (width 0.4) (layer "B.Cu") (net 132))
-  (segment (start 109.202 120.954) (end 115.212 126.964) (width 0.4) (layer "B.Cu") (net 132))
+  (segment (start 113.902 126.964) (end 108.902 121.964) (width 0.4) (layer "B.Cu") (net 132))
+  (segment (start 115.212 126.964) (end 113.902 126.964) (width 0.4) (layer "B.Cu") (net 132))
+  (segment (start 114.602 116.514) (end 116.822 114.294) (width 0.4) (layer "B.Cu") (net 132))
+  (segment (start 116.822 114.294) (end 116.822 112.244) (width 0.4) (layer "B.Cu") (net 132))
+  (segment (start 108.902 121.964) (end 105.952 121.964) (width 0.4) (layer "B.Cu") (net 132))
+  (segment (start 106.752 116.514) (end 114.602 116.514) (width 0.4) (layer "B.Cu") (net 132))
+  (segment (start 105.952 117.314) (end 106.752 116.514) (width 0.4) (layer "B.Cu") (net 132))
+  (segment (start 105.952 121.964) (end 105.952 117.314) (width 0.4) (layer "B.Cu") (net 132))
   (segment (start 115.212 129.964) (end 115.212 126.964) (width 0.4) (layer "B.Cu") (net 132))
   (segment (start 81.502 143.964) (end 81.502 134.694) (width 0.4) (layer "F.Cu") (net 133))
@@
     (connect_pads (clearance 0.508))
     (min_thickness 0.254) (filled_areas_thickness no)
-    (fill (thermal_gap 0.508) (thermal_bridge_width 0.508))
+    (fill yes (thermal_gap 0.508) (thermal_bridge_width 0.508))
     (polygon
       (pts
@@
     (connect_pads (clearance 0.508))
     (min_thickness 0.254) (filled_areas_thickness no)
-    (fill (thermal_gap 0.508) (thermal_bridge_width 0.508))
+    (fill yes (thermal_gap 0.508) (thermal_bridge_width 0.508))
     (polygon
       (pts
