File: CV_Trigger_Sequencer/DrumSequencer/DrumSequencer.kicad_sch (KiCad schematic)
At the start: 171 parts, among them J1 Conn_01x06_Male, J2 Conn_01x06_Male, Q1 NDT3055L, Q19 BC547, Q2 BC547, Q20 BC547, Q21 BC547, Q22 BC547, Q23 BC547, Q24 BC547, Q25 BC547, Q26 BC547, Q27 BC547, Q28 BC547, Q3 BC557, Q8 BC547, SW2 SW_Push, U1 TL074, U10 Switch, U11 Switch, U12 Switch, U13 Switch, U14 Switch, U15 Switch, U16 Aux_flush, U16 SP3T, U17 Aux_flush, U17 SP3T, U18 Aux_flush, U18 SP3T, U19 Aux_flush, U19 SP3T, U2 ATmega328-P, U2 TL072, U20 LM7805_TO220, U20 SP3T, U21 SP3T, U22 SP3T, U23 SP3T, U24 Aux_flush, U25 Aux_flush, U26 Aux_flush, U3 TL074, U4 Aux_flush, U6 Aux_flush, U7 Aux_flush, U8 Switch, U9 Switch, Y1 Crystal

Commit message: Add files via upload
Connections:
- net IN1: now also U2.25 (PC2); no longer U2.1 (~{RESET}/PC6)
Other:
- moved on the sheet: C1, C2, C3, C4, C5, C6, C7, C8, D10, D11, D12, D13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
