File: DoubleDelay/DoubleDelay.kicad_pcb (KiCad board)
At the start: 2 copper layers, 114 x 128 mm, 83 parts, among them J1 Conn_01x06_Male, J2 Conn_01x06_Male, J3 Conn_01x15_Male, J4 Conn_01x15_Male, Q1 BC547, Q2 BC547, U1 Aux_flush, U10 Aux_flush, U2 TL074, U3 PT2399, U4 Aux_flush, U5 LM7805_TO220, U6 Aux_flush, U7 Switch, U9 PT2399

Commit message: Add files via upload
Parts:
- removed C26: C, Capacitor_THT:C_Axial_L3.8mm_D2.6mm_P7.50mm_Horizontal
- removed D2: LED, LED_THT:LED_D5.0mm
- removed Q1: BC547, Package_TO_SOT_THT:TO-92_Inline_Wide
- removed R13, R15, R38: R, Resistor_THT:R_Axial_DIN0207_L6.3mm_D2.5mm_P7.62mm_Horizontal
- added ?: , clipboard:c0182654-ed92-4dac-bfe7-a251b8662b05, F.Cu at (176.4, 48.9)
- added ?: , clipboard:c0182654-ed92-4dac-bfe7-a251b8662b05, F.Cu at (202.3, 132.5)
- added ?: , clipboard:c0182654-ed92-4dac-bfe7-a251b8662b05, F.Cu at (208.0, 51.0)
- added ?: , clipboard:c0182654-ed92-4dac-bfe7-a251b8662b05, F.Cu at (183.3, 65.5)
- added ?: , clipboard:c0182654-ed92-4dac-bfe7-a251b8662b05, F.Cu at (183.1, 117.0)
- added ?: , clipboard:c0182654-ed92-4dac-bfe7-a251b8662b05, F.Cu at (207.8, 140.7)
- added ?: , clipboard:c0182654-ed92-4dac-bfe7-a251b8662b05, F.Cu at (208.0, 109.3)
- added ?: , clipboard:c0182654-ed92-4dac-bfe7-a251b8662b05, F.Cu at (208.1, 78.2)
- added ?: , clipboard:c0182654-ed92-4dac-bfe7-a251b8662b05, F.Cu at (183.6, 90.2)
- added ?: , clipboard:c0182654-ed92-4dac-bfe7-a251b8662b05, F.Cu at (189.1, 48.9)
- added ?: , clipboard:c0182654-ed92-4dac-bfe7-a251b8662b05, F.Cu at (214.2, 132.6)
- added ?: , clipboard:c0182654-ed92-4dac-bfe7-a251b8662b05, F.Cu at (181.8, 141.6)
- added REF**: MountingHole_3.2mm_M3, MountingHole:MountingHole_3.2mm_M3, F.Cu at (211.5, 31.7)
- added REF**: MountingHole_3.2mm_M3, MountingHole:MountingHole_3.2mm_M3, F.Cu at (181.0, 31.7)
- added REF**: MountingHole_3.2mm_M3, MountingHole:MountingHole_3.2mm_M3, F.Cu at (181.0, 154.2)
- added REF**: MountingHole_3.2mm_M3, MountingHole:MountingHole_3.2mm_M3, F.Cu at (211.5, 154.2)
- C1, C15, C17, C18, C20, C22, C3, C4, C7, C9: value C -> 100n
- C10, C21, C23, C8: value C -> 500p
- C11, C13, C14, C19, C5: value C_Polarized -> 1u
- C16, C2: value C_Polarized -> 47u
- R10, R11, R12, R32, R34, R35, R36, R8: value R -> 10k
- R16, R26: value R -> 47k
- R17, R18, R21, R22, R24, R27, R28, R30, R31, R4, R5, R6, R7: value R -> 100k
- R23, R29, R3, R9: value R -> 1k
- R33: value R -> 2k2
- R37, R39: value R -> 0R
- U1, U10, U4, U6: footprint Library:aux_flush -> Library:3mm5 Mono Aux
- moved J3 94.5 mm to (123.2, 81.3)
- moved R29 62.2 mm to (138.2, 134.2), turned to 180 degrees
- moved R31 37.4 mm to (138.1, 126.8), turned to 180 degrees
- moved Q2 29.5 mm to (148.7, 124.7), turned to -90 degrees
- moved R27 27.7 mm to (129.5, 116.2)
- moved R21 15.8 mm to (148.8, 110.5), turned to 90 degrees
- moved R3 15.3 mm to (87.5, 130.5)
- moved C1 15.3 mm to (89.0, 122.3)
- moved C15 15.3 mm to (85.2, 55.6)
- moved C18 15.3 mm to (82.3, 78.3)
- moved C19 15.3 mm to (103.7, 106.8)
- moved C2 15.3 mm to (87.0, 126.8)
- moved C21 15.3 mm to (104.2, 56.7)
- moved C25 15.3 mm to (104.2, 69.7)
- moved C5 15.3 mm to (92.7, 80.6)
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Connections:
- C10 pad 1: Net-(C10-Pad1) -> Net-(U3-LPF2-OUT)
- C11 pad 1: Net-(C11-Pad1) -> Net-(U3-LPF2-OUT)
- R12 pad 1: Net-(C10-Pad1) -> Net-(U3-LPF2-OUT)
- U3 pad 14: Net-(C10-Pad1) -> Net-(U3-LPF2-OUT)
Routing:
- net DOUT2: track 0.00 -> 124.3 mm, vias 0 -> 1
- net X1: track 55.1 -> 152.3 mm, vias 0 -> 3
- net VGND4: track 12.4 -> 104.4 mm, vias 0 -> 3
- net DOUT1: track 0.00 -> 89.6 mm
- net -12V: track 0.00 -> 85.2 mm
- net +5V: track 28.5 -> 105.4 mm
- net VGND3: track 0.00 -> 68.2 mm, vias 0 -> 3
- net Net-(C13-Pad2): track 0.00 -> 67.3 mm, vias 0 -> 1
- net VCO2: track 6.42 -> 50.5 mm
- net VGND1: track 24.3 -> 63.4 mm
- net Net-(U6-Pad1): track 0.00 -> 34.3 mm
- net Net-(U3-LPF2-OUT): track 0.00 -> 33.4 mm
- net Net-(D3-K): track 0.00 -> 32.4 mm
- net VGND2: track 17.8 -> 48.7 mm
- net Net-(R29-Pad1): track 0.00 -> 29.0 mm
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- added copper zone on F.Cu, net +12V
- added copper zone on B.Cu, net GND
Other:
- board size 114 x 128 mm -> 147.6 x 128 mm
