File: DoubleDelay/DoubleDelay.kicad_sch (KiCad schematic)
At the start: 82 parts, among them J1 Conn_01x06_Male, J2 Conn_01x06_Male, J3 Conn_01x15_Male, J4 Conn_01x15_Male, Q1 BC547, Q2 BC547, U1 Aux_flush, U10 Aux_flush, U2 TL074, U3 PT2399, U4 Aux_flush, U5 LM7805_TO220, U6 Aux_flush, U7 Switch, U9 PT2399

Commit message: Add files via upload
Parts:
- removed C26: C, Capacitor_THT:C_Axial_L3.8mm_D2.6mm_P7.50mm_Horizontal, symbol Device:C
- removed D2: LED, LED_THT:LED_D5.0mm, symbol Device:LED
- removed Q1: BC547, Package_TO_SOT_THT:TO-92_Inline_Wide, symbol Transistor_BJT:BC547
- removed R13, R15: R, Resistor_THT:R_Axial_DIN0207_L6.3mm_D2.5mm_P7.62mm_Horizontal, symbol Device:R
- C1, C15, C17, C18, C20, C22, C3, C4, C7, C9: value C -> 100n
- C10, C21, C23, C8: value C -> 500p
- C11, C13, C14, C19, C24, C25, C5, C6: value C_Polarized -> 1u
- C16, C2: value C_Polarized -> 4u7
- R10, R11, R12, R32, R34, R35, R36, R8: value R -> 10k
- R16, R26: value R -> 47k
- R17, R18, R21, R22, R24, R27, R28, R30, R31, R4, R5, R6, R7: value R -> 100k
- R23, R29, R3, R9: value R -> 1k
- R33: value R -> 2k2
- R37, R39: value R -> 0R
- U1, U10, U4, U6: footprint Library:aux_flush -> Library:3mm5 Mono Aux
Other:
- title: (none) -> DoubleDelay by github.com/Fihdi
