File: utility/utility.kicad_pcb (KiCad board)
At the start: 2 copper layers, 147.4 x 128 mm, 102 parts, among them J1 Conn_01x06_Male, J2 Conn_01x06_Male, J3 Conn_01x06_Male, J4 Conn_01x06_Male, J5 Conn_01x06_Male, J6 Conn_01x06_Male, J7 Conn_01x06_Male, Q1 BC547, Q2 BC547, U1 Aux_flush, U10 Aux_flush, U11 Aux_flush, U12 TL072, U13 Aux_flush, U14 Aux_flush, U15 Aux_flush, U16 TL072, U17 TL072, U18 TL072, U19 Aux_flush, U2 Aux_flush, U20 Aux_flush, U21 Aux_flush, U22 Aux_flush, U23 Aux_flush, U24 Aux_flush, U25 Aux_flush, U26 Aux_flush, U3 TL074, U4 LM2907, U5 Aux_flush, U6 Aux_flush, U7 Aux_flush, U8 Aux_flush, U9 Aux_flush

Commit message: Add files via upload
Minor improvements
Routing:
- net -12V: track 476.9 -> 540.8 mm, vias 0 -> 3
