File: utility/utility.kicad_sch (KiCad schematic)
At the start: 92 parts, among them J1 Conn_01x06_Male, J2 Conn_01x06_Male, J3 Conn_01x06_Male, J4 Conn_01x06_Male, J5 Conn_01x06_Male, J6 Conn_01x06_Male, J7 Conn_01x06_Male, Q1 BC547, Q2 BC547, U1 Aux_flush, U10 Aux_flush, U11 Aux_flush, U12 TL072, U13 Aux_flush, U14 Aux_flush, U15 Aux_flush, U16 TL072, U17 TL072, U18 TL072, U19 Aux_flush, U2 Aux_flush, U20 Aux_flush, U21 Aux_flush, U22 Aux_flush, U23 Aux_flush, U24 Aux_flush, U25 Aux_flush, U26 Aux_flush, U3 TL074, U4 LM2907, U5 Aux_flush, U6 Aux_flush, U7 Aux_flush, U8 Aux_flush, U9 Aux_flush

Commit message: Add files via upload
Minor improvements
Parts:
- C1, C2: value C -> 100n
- C3: value C -> 1u
- R1, R10, R12, R13, R18, R19, R3, R5: value R -> 50k
- R11, R15, R25, R33, R37, R6: value R -> 1k
- R14, R16, R7: value R -> 10k
- R17, R38, R39, R8: value R -> 2k2
- R2: value AlpsPot -> 100k
- R20, R9: value AlpsPot -> 1M
- R23, R24, R26, R27, R28, R29, R31, R32, R35, R36, R4, R40, R41, R42, R43: value R -> 100k
Other:
- title: (none) -> Utility by github.com/Fihdi
- moved on the sheet: J1, J2, J3, J4, J5, J6, J7, U3B
