File: AXOR/AXOR.kicad_pcb (KiCad board)
At the start: 2 copper layers, 118.5 x 128.5 mm, 58 parts, among them J1 Conn_01x06_Pin, J2 Conn_01x12_Pin, J3 Conn_01x12_Pin, SW1 SW_SPDT, SW2 SW_SPDT, U1 Aux_flush, U10 Aux_flush, U11 TL074, U12 Aux_flush, U13 Aux_flush, U14 Aux_flush, U2 Aux_flush, U3 Aux_flush, U7 Aux_flush, U9 LM13700

Commit message: Add files via upload
Parts:
- added Q1: BC557, Package_TO_SOT_THT:TO-92_Inline_Wide, F.Cu at (198.4, 73.1)
- added Q2: BC557, Package_TO_SOT_THT:TO-92_Inline_Wide, F.Cu at (193.6, 70.4)
Connections:
- R22 pad 2: Net-(R22-Pad2) -> Net-(Q2-E)
- R4 pad 2: Net-(R4-Pad2) -> Net-(Q1-E)
- U9 pad 1: Net-(R22-Pad2) -> Net-(Q2-C)
- U9 pad 16: Net-(R4-Pad2) -> Net-(Q1-C)
Routing:
- net Net-(Q2-C): track 0.00 -> 7.33 mm
- net IN1: track 163.5 -> 170.8 mm
- net Net-(Q2-E): track 0.00 -> 7.01 mm
- net -12V: track 83.1 -> 88.9 mm
- net Net-(Q1-C): track 0.00 -> 4.72 mm
- net Net-(Q1-E): track 0.00 -> 4.55 mm
- net Net-(R22-Pad2): track 3.06 -> 0.00 mm
- net Net-(R4-Pad2): track 2.91 -> 0.00 mm
Other:
- outline, holes or cut-outs redrawn
