File: SimpleSampler/SimpleSampler.kicad_pcb (KiCad board)
At the start: 2 copper layers, 96.2 x 128 mm, 49 parts, among them J1 Conn_01x06_Pin, J2 Conn_01x10_Pin, J24 Conn_01x10_Pin, J3 Conn_01x01_Pin, J4 Conn_01x01_Pin, Q1 BC547, Q2 BC547, Q3 BC547, SW1 RotaryEncoder_Switch, SW2 SW_Push, U1 TL072, U2 Aux_flush, U4 Aux_flush, U5 Aux_flush, U6 Switch, U7 Aux_flush

Commit message: Add files via upload
Parts:
- R1, R2, R4, R5: value R -> 100k
- R10, R12, R15, R16, R7, R8, R9: value R -> 10k
- R11: value R -> 560R
- R13: value R -> 330R to 1k
- R3: value R -> 200k
- R6: value R -> 4k7
- SW2: footprint Connector_PinHeader_2.54mm:PinHeader_1x02_P2.54mm_Vertical -> Library:PushButton
- moved SW2 9.19 mm to (157.2, 50.8), turned to 0 degrees
Routing:
- net Net-(R10-Pad2): track 2.49 -> 8.72 mm
- net LENGTH: track 102.8 -> 103.4 mm
- net CV: track 136.5 -> 137.1 mm
Other:
- board text added: "SPEED"
- board text added: "TRIGGER"
- board text removed: "PITCH"
- board text removed: "TRG"

Commit message: Add files via upload
Parts:
- removed Q2: BC547, Package_TO_SOT_THT:TO-92_Inline_Wide
- removed R10, R12: 10k, Resistor_THT:R_Axial_DIN0207_L6.3mm_D2.5mm_P7.62mm_Horizontal
- removed R13: 330R to 1k, Resistor_THT:R_Axial_DIN0207_L6.3mm_D2.5mm_P7.62mm_Horizontal
- removed U5: Aux_flush, Library:3mm5 Mono Aux
- added J6: Micro_SD_Card, Connector_Card:microSD_HC_Molex_47219-2001, F.Cu at (176.2, 62.2)
- added R14: ~, Resistor_THT:R_Axial_DIN0207_L6.3mm_D2.5mm_P7.62mm_Horizontal, F.Cu at (193.0, 132.9)
- added R17: ~, Resistor_THT:R_Axial_DIN0207_L6.3mm_D2.5mm_P7.62mm_Horizontal, F.Cu at (189.5, 140.6)
- added R18: ~, Resistor_THT:R_Axial_DIN0207_L6.3mm_D2.5mm_P7.62mm_Horizontal, F.Cu at (186.0, 132.9)
- added R19: ~, Resistor_THT:R_Axial_DIN0207_L6.3mm_D2.5mm_P7.62mm_Horizontal, F.Cu at (159.5, 142.6)
- added U3: Aux_flush, Library:3mm5 Mono Aux, F.Cu at (150.2, 138.5)
- R11: value 560R -> 1k
- U1: value TL072 -> TL074; footprint Package_DIP:DIP-8_W7.62mm -> Package_DIP:DIP-14_W7.62mm
- moved U1 22.2 mm to (201.9, 122.2), turned to -90 degrees
- moved R5 16.9 mm to (198.0, 140.6)
- moved R6 16.9 mm to (201.5, 132.9)
- moved A1 10.6 mm to (187.1, 56.5)
- moved J1 10.6 mm to (207.6, 69.4)
- moved J3 10.6 mm to (181.6, 137.1)
- moved R2 10.6 mm to (192.8, 111.1)
- moved R4 6.48 mm to (182.0, 118.4)
- moved J24 1.05 mm to (170.0, 92.8)
Connections:
- A1 pad 2: unconnected-(A1-SD_DATA_3-Pad2) -> D3
- A1 pad 3: unconnected-(A1-SD_DATA_2-Pad3) -> D2
- A1 pad 4: unconnected-(A1-SD_DATA_1-Pad4) -> D1
- A1 pad 5: unconnected-(A1-SD_DATA_0-Pad5) -> D0
- A1 pad 6: unconnected-(A1-SD_CMD-Pad6) -> SCD
- A1 pad 7: unconnected-(A1-SD_CLK-Pad7) -> SCLK
- D1 pad 2: +3V3 -> LED
- J2 pad 9: AUD -> OUT
- J24 pad 9: AUD -> OUT
- R11 pad 1: Net-(Q2-C) -> GND
- R4 pad 2: Net-(U1A--) -> Net-(U1B--)
- R5 pad 1: Net-(U1A--) -> Net-(U1B--)
- SW2 pad 1: +3V3 -> PLAY
- SW2 pad 2: Net-(R10-Pad2) -> GND
- U1 pad 1: Net-(R5-Pad2) -> Net-(R2-Pad2)
- U1 pad 2: Net-(U1A--) -> SUM
- U1 pad 4: -12V -> +12V
- U1 pad 6: SUM -> Net-(U1B--)
- U1 pad 7: Net-(R2-Pad2) -> Net-(R5-Pad2)
- U1 pad 8: +12V -> OUT
Routing:
- net OUT: track 0.00 -> 72.5 mm
- net Net-(U1B--): track 0.00 -> 36.3 mm
- net Net-(R5-Pad2): track 6.72 -> 37.8 mm
- net AUD: track 98.1 -> 71.5 mm, vias 1 -> 3
- net Net-(U1A--): track 25.8 -> 0.00 mm
- net PLAY: track 98.9 -> 118.9 mm
- net D2: track 0.00 -> 19.9 mm
- net SCLK: track 0.00 -> 19.2 mm
- net LED: track 80.3 -> 99.4 mm
- net SCD: track 0.00 -> 18.9 mm, vias 0 -> 1
- net D3: track 0.00 -> 16.1 mm, vias 0 -> 1
- net Net-(Q2-B): track 15.7 -> 0.00 mm
- net D0: track 0.00 -> 15.0 mm
- net SUM: track 74.9 -> 85.6 mm
- net LENGTH: track 103.4 -> 113.2 mm
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Other:
- board size 96.2 x 128 mm -> 107.2 x 128 mm
