File: SimpleSampler/SimpleSampler.kicad_sch (KiCad schematic)
At the start: 38 parts, among them J1 Conn_01x06_Pin, J2 Conn_01x10_Pin, J24 Conn_01x10_Pin, J3 Conn_01x01_Pin, J4 Conn_01x01_Pin, Q1 BC547, Q2 BC547, Q3 BC547, SW1 RotaryEncoder_Switch, SW2 SW_Push, U1 TL072, U2 Aux_flush, U4 Aux_flush, U5 Aux_flush, U6 Switch, U7 Aux_flush

Commit message: Add files via upload
Parts:
- SW2: footprint Connector_PinHeader_2.54mm:PinHeader_1x02_P2.54mm_Vertical -> Library:PushButton
Changed lines of the file:
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@@
       (effects (font (size 1.27 1.27)))
     )
-    (property "Footprint" "Connector_PinHeader_2.54mm:PinHeader_1x02_P2.54mm_Vertical" (at 48.26 104.14 0)
+    (property "Footprint" "Library:PushButton" (at 48.26 104.14 0)
       (effects (font (size 1.27 1.27)) hide)
     )

Commit message: Add files via upload
Parts:
- removed Q2: BC547, Package_TO_SOT_THT:TO-92_Inline_Wide, symbol Transistor_BJT:BC547
- removed R10, R12: 10k, Resistor_THT:R_Axial_DIN0207_L6.3mm_D2.5mm_P7.62mm_Horizontal, symbol Device:R
- removed R13: 330R to 1k, Resistor_THT:R_Axial_DIN0207_L6.3mm_D2.5mm_P7.62mm_Horizontal, symbol Device:R
- removed U1: TL072, Package_DIP:DIP-8_W7.62mm, symbol Amplifier_Operational:TL072
- removed U5: Aux_flush, Library:3mm5 Mono Aux, symbol HEJ:Aux_flush
- added J6: Micro_SD_Card, Connector_Card:microSD_HC_Molex_47219-2001, symbol Connector:Micro_SD_Card
- added R14, R17, R18, R19: ~, Resistor_THT:R_Axial_DIN0207_L6.3mm_D2.5mm_P7.62mm_Horizontal, symbol Device:R
- added U1: TL074, Package_DIP:DIP-14_W7.62mm, symbol Amplifier_Operational:TL074
- added U3: Aux_flush, Library:3mm5 Mono Aux, symbol HEJ:Aux_flush
- R11: value 560R -> 1k
Connections:
- net +12V: now also U1.4 (V+)
- net +3V3: now also J6.4 (VDD); no longer D1.2 (A), SW2.1
- net -12V: now also U1.11 (V-)
- net AUD: now also R14.2; no longer J2.9 (Pin_9), J24.9 (Pin_9)
- net GND: now also R11.1, SW2.2, J6.6 (VSS), U1.10 (+), U1.3 (+), U1.5 (+)
- net LED: now also D1.2 (A)
- net PLAY: now also SW2.1
- net SUM: now also U1.2 (-)
- net at R4.2, R5.1: now also U1.6 (-)
- net at R5.2, R6.1: now also U1.7
- net D3: now reaches A1.2 (SD_DATA_3)
- net D3: now also J6.2 (DAT3/CD)
- net D2: now reaches A1.3 (SD_DATA_2)
- net D2: now also J6.1 (DAT2)
- net D1: now reaches A1.4 (SD_DATA_1)
- net D1: now also J6.8 (DAT1)
- net D0: now reaches A1.5 (SD_DATA_0)
- net D0: now also J6.7 (DAT0)
- net SCD: now reaches A1.6 (SD_CMD)
- net SCD: now also J6.3 (CMD)
- net SCLK: now reaches A1.7 (SD_CLK)
- net SCLK: now also J6.5 (CLK)
- net at R2.2, R4.1: now also U1.1
- new net: R19.1, U3.1
- new net: R17.1, R18.2
- new net: R14.1, R17.2, U1.9 (-)
- new net OUT: J2.9 (Pin_9), J24.9 (Pin_9), R18.1, R19.2, U1.8
- no-connect marks 28 -> 23
Other:
- note added: "Daisy"
- note added: "SD Card"
- title: (none) -> Samples by github.com/Fihdi
- moved on the sheet: A1, D1, D4, D5, Q1, Q3, R11, R15, R16, R7, R8, R9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
