File: TRIVCO/TRIVCO.kicad_pcb (KiCad board)
At the start: 2 copper layers, 102.9 x 128.2 mm, 53 parts, among them J1 Conn_01x06_Pin, J2 Conn_01x10_Pin, J4 Conn_01x10_Pin, Q1 BC557, Q2 BC557, Q3 BC547, U1 TL074, U10 Aux_flush, U2 LM13700, U3 Switch, U4 TL074, U5 Aux_flush, U6 Aux_flush, U7 Aux_flush, U8 Aux_flush, U9 Aux_flush

Commit message: Add files via upload
Parts:
- added REF**: MountingHole_3.2mm_M3, MountingHole:MountingHole_3.2mm_M3, F.Cu at (74.9, 55.2)
- added REF**: MountingHole_3.2mm_M3, MountingHole:MountingHole_3.2mm_M3, F.Cu at (46.6, 144.0)
- added REF**: MountingHole_3.2mm_M3, MountingHole:MountingHole_3.2mm_M3, F.Cu at (89.4, 55.2)
- added REF**: MountingHole_3.2mm_M3, MountingHole:MountingHole_3.2mm_M3, F.Cu at (88.8, 144.1)
- added REF**: MountingHole_3.2mm_M3, MountingHole:MountingHole_3.2mm_M3, F.Cu at (70.2, 119.1)
- added REF**: MountingHole_3.2mm_M3, MountingHole:MountingHole_3.2mm_M3, F.Cu at (50.9, 99.1)
- added REF**: MountingHole_3.2mm_M3, MountingHole:MountingHole_3.2mm_M3, F.Cu at (62.5, 19.0)
- added REF**: MountingHole_3.2mm_M3, MountingHole:MountingHole_3.2mm_M3, F.Cu at (92.0, 23.5)
- added REF**: MountingHole_3.2mm_M3, MountingHole:MountingHole_3.2mm_M3, F.Cu at (88.0, 118.9)
- added REF**: MountingHole_3.2mm_M3, MountingHole:MountingHole_3.2mm_M3, F.Cu at (60.6, 144.0)
- added REF**: MountingHole_3.2mm_M3, MountingHole:MountingHole_3.2mm_M3, F.Cu at (50.8, 75.5)
- added REF**: MountingHole_3.2mm_M3, MountingHole:MountingHole_3.2mm_M3, F.Cu at (74.6, 144.1)
- U10, U5, U6, U7, U8, U9: footprint Library:aux_flush -> Library:3mm5 Mono Aux
- moved REF** 74.1 mm to (52.0, 55.1)
- moved REF** 72.4 mm to (89.6, 161.0)
- moved REF** 72.4 mm to (89.6, 38.5)
- moved REF** 72.4 mm to (49.0, 38.5)
- moved REF** 72.4 mm to (49.0, 161.0)
- moved U3 8.77 mm to (129.3, 70.4)
- moved Q2 1.60 mm to (213.7, 78.5)
- moved R16 1.60 mm to (175.8, 119.0)
- moved R3 1.60 mm to (197.3, 116.2)
- moved R8 1.60 mm to (196.8, 77.0)
- moved U1 1.60 mm to (188.5, 100.7)
- moved C1 1.60 mm to (204.4, 106.2)
- moved C3 1.60 mm to (210.9, 126.5)
- moved J1 1.60 mm to (217.1, 116.4)
- moved J4 1.60 mm to (175.4, 89.0)
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Routing:
- net CAP: track 148.1 -> 144.1 mm
- net Net-(D1-A): track 7.02 -> 9.84 mm
- net SYN: track 180.1 -> 179.0 mm
- net Net-(R17-Pad1): track 19.4 -> 18.7 mm
- net Net-(R6-E): track 26.3 -> 25.7 mm
- net Net-(R25-E): track 35.1 -> 34.5 mm
- net Net-(R12-Pad1): track 8.50 -> 7.92 mm
Other:
- board size 102.9 x 128.2 mm -> 179.9 x 128.2 mm
