File: TRIVCO/TRIVCO.kicad_sch (KiCad schematic)
At the start: 48 parts, among them J1 Conn_01x06_Pin, J2 Conn_01x10_Pin, J4 Conn_01x10_Pin, Q1 BC557, Q2 BC557, Q3 BC547, U1 TL074, U10 Aux_flush, U2 LM13700, U3 Switch, U4 TL074, U5 Aux_flush, U6 Aux_flush, U7 Aux_flush, U8 Aux_flush, U9 Aux_flush

Commit message: Add files via upload
Parts:
- U10, U5, U6, U7, U8, U9: footprint Library:aux_flush -> Library:3mm5 Mono Aux
