File: VCF/VCF.kicad_sch (KiCad schematic)
At the start: 52 parts, among them J1 Conn_01x10_Pin, J2 Conn_01x10_Pin, J3 Conn_01x06_Pin, Q1 BC557, Q2 BC557, Q3 BC547, U1 Aux_flush, U10 Aux_flush, U11 Aux_flush, U2 Aux_flush, U3 TL074, U4 TL072, U5 LM13700, U6 Aux_flush, U7 Aux_flush, U9 Aux_flush

Commit message: Add files via upload
Parts:
- R21: footprint 1k -> Resistor_THT:R_Axial_DIN0207_L6.3mm_D2.5mm_P10.16mm_Horizontal
- U1, U10, U11, U2, U6, U7, U9: footprint Library:aux_flush -> Library:3mm5 Mono Aux
Changed lines of the file:
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@@
       (effects (font (size 1.27 1.27)) hide)
     )
+    (pin "1")
+    (pin "2")
     (pin "3")
+    (pin "4")
     (pin "5")
-    (pin "1")
-    (pin "4")
-    (pin "2")
     (pin "6")
     (instances
@@
       (effects (font (size 1.27 1.27)) hide)
     )
-    (property "Footprint" "Library:aux_flush" (at 42.545 54.737 0)
+    (property "Footprint" "Library:3mm5 Mono Aux" (at 42.545 54.737 0)
       (effects (font (size 1.27 1.27)) hide)
     )
@@
       (effects (font (size 1.27 1.27)) hide)
     )
-    (property "Footprint" "Library:aux_flush" (at 268.605 104.267 0)
+    (property "Footprint" "Library:3mm5 Mono Aux" (at 268.605 104.267 0)
       (effects (font (size 1.27 1.27)) hide)
     )
@@
       (effects (font (size 1.27 1.27)) hide)
     )
-    (property "Footprint" "Library:aux_flush" (at 37.338 127.762 0)
+    (property "Footprint" "Library:3mm5 Mono Aux" (at 37.338 127.762 0)
       (effects (font (size 1.27 1.27)) hide)
     )
@@
       (effects (font (size 1.27 1.27)) hide)
     )
-    (property "Footprint" "Library:aux_flush" (at 269.113 57.658 0)
+    (property "Footprint" "Library:3mm5 Mono Aux" (at 269.113 57.658 0)
       (effects (font (size 1.27 1.27)) hide)
     )
@@
       (effects (font (size 1.27 1.27)) (justify left) hide)
     )
+    (pin "1")
     (pin "2")
     (pin "3")
-    (pin "1")
     (instances
       (project "VCF"
@@
       (effects (font (size 1.27 1.27)) hide)
     )
+    (pin "1")
     (pin "10")
+    (pin "2")
     (pin "3")
+    (pin "4")
+    (pin "5")
+    (pin "6")
     (pin "7")
+    (pin "8")
     (pin "9")
-    (pin "8")
-    (pin "4")
-    (pin "1")
-    (pin "2")
-    (pin "6")
-    (pin "5")
     (instances
       (project "VCF"
@@
   (symbol (lib_id "HEJ:Aux_flush") (at 37.338 119.253 0) (unit 1)
     (in_bom yes) (on_board yes) (dnp no) (fields_autoplaced)
-    (property "Reference" "U7" (at 37.3126 114.681 0)
+    (property "Reference" "U7" (at 37.3126 115.57 0)
       (effects (font (size 1.27 1.27)))
     )
@@
       (effects (font (size 1.27 1.27)) hide)
     )
-    (property "Footprint" "Library:aux_flush" (at 37.338 119.253 0)
+    (property "Footprint" "Library:3mm5 Mono Aux" (at 37.338 119.253 0)
       (effects (font (size 1.27 1.27)) hide)
     )
@@
       (effects (font (size 1.27 1.27)) hide)
     )
-    (property "Footprint" "Library:aux_flush" (at 42.418 66.04 0)
+    (property "Footprint" "Library:3mm5 Mono Aux" (at 42.418 66.04 0)
       (effects (font (size 1.27 1.27)) hide)
     )
@@
       (effects (font (size 1.27 1.27)) hide)
     )
+    (pin "1")
     (pin "10")
+    (pin "2")
     (pin "3")
+    (pin "4")
+    (pin "5")
+    (pin "6")
     (pin "7")
+    (pin "8")
     (pin "9")
-    (pin "8")
-    (pin "4")
-    (pin "1")
-    (pin "2")
-    (pin "6")
-    (pin "5")
     (instances
       (project "VCF"
@@
   (symbol (lib_id "Device:R") (at 152.908 62.357 90) (unit 1)
     (in_bom yes) (on_board yes) (dnp no) (fields_autoplaced)
-    (property "Reference" "R19" (at 152.908 56.007 90)
-      (effects (font (size 1.27 1.27)))
-    )
-    (property "Value" "200k" (at 152.908 58.547 90)
+    (property "Reference" "R19" (at 152.908 55.88 90)
+      (effects (font (size 1.27 1.27)))
+    )
+    (property "Value" "200k" (at 152.908 58.42 90)
       (effects (font (size 1.27 1.27)))
     )
@@
       (effects (font (size 1.27 1.27)) (justify right))
     )
-    (property "Footprint" "1k" (at 162.941 67.31 90)
+    (property "Footprint" "Resistor_THT:R_Axial_DIN0207_L6.3mm_D2.5mm_P10.16mm_Horizontal" (at 162.941 67.31 90)
       (effects (font (size 1.27 1.27)) hide)
     )
@@
       (effects (font (size 1.27 1.27)) hide)
     )
-    (property "Footprint" "Library:aux_flush" (at 268.732 81.153 0)
-      (effects (font (size 1.27 1.27)) hide)
-    )
+    (property "Footprint" "Library:3mm5 Mono Aux" (at 268.732 81.153 0)
+      (effects (font (size 1.27 1.27)) hide)
+    )
