File: Switch/Switch.kicad_sch (KiCad schematic)
At the start: 61 parts, among them J1 Conn_01x14_Pin, J2 Conn_01x14_Pin, J3 Conn_01x06_Pin, Q1 BC547, Q2 BC547, Q3 BC547, Q4 BC547, U1 TL074, U11 Aux_flush, U12 Aux_flush, U13 Aux_flush, U14 Aux_flush, U15 Aux_flush, U16 Aux_flush, U2 CD4066BE, U3 TL074, U4 Aux_flush, U5 Aux_flush, U6 Aux_flush, U7 Aux_flush, U8 Aux_flush, U9 Aux_flush

Commit message: Add files via upload
Parts:
- U11, U12, U13, U14, U15, U16, U4, U5, U6, U7, U8, U9: footprint Library:aux_flush -> Library:3mm5 Mono Aux
- U3: footprint (none) -> Package_DIP:DIP-14_W7.62mm_Socket
Changed lines of the file:
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@@
       (effects (font (size 1.27 1.27)) hide)
     )
-    (property "Footprint" "Library:aux_flush" (at 128.27 136.525 0)
+    (property "Footprint" "Library:3mm5 Mono Aux" (at 128.27 136.525 0)
       (effects (font (size 1.27 1.27)) hide)
     )
@@
       (effects (font (size 1.27 1.27)) (justify right))
     )
-    (property "Footprint" "" (at 252.095 61.595 0)
+    (property "Footprint" "Package_DIP:DIP-14_W7.62mm_Socket" (at 252.095 61.595 0)
       (effects (font (size 1.27 1.27)) hide)
     )
@@
       (effects (font (size 1.27 1.27)) hide)
     )
-    (property "Footprint" "Library:aux_flush" (at 87.63 142.24 0)
+    (property "Footprint" "Library:3mm5 Mono Aux" (at 87.63 142.24 0)
       (effects (font (size 1.27 1.27)) hide)
     )
@@
       (effects (font (size 1.27 1.27)) hide)
     )
-    (property "Footprint" "Library:aux_flush" (at 259.715 106.045 0)
+    (property "Footprint" "Library:3mm5 Mono Aux" (at 259.715 106.045 0)
       (effects (font (size 1.27 1.27)) hide)
     )
@@
       (effects (font (size 1.27 1.27)) hide)
     )
-    (property "Footprint" "Library:aux_flush" (at 258.445 140.335 0)
+    (property "Footprint" "Library:3mm5 Mono Aux" (at 258.445 140.335 0)
       (effects (font (size 1.27 1.27)) hide)
     )
@@
       (effects (font (size 1.27 1.27)) hide)
     )
-    (property "Footprint" "Library:aux_flush" (at 67.945 40.64 0)
+    (property "Footprint" "Library:3mm5 Mono Aux" (at 67.945 40.64 0)
       (effects (font (size 1.27 1.27)) hide)
     )
@@
       (effects (font (size 1.27 1.27)) hide)
     )
-    (property "Footprint" "Library:aux_flush" (at 177.8 45.72 0)
+    (property "Footprint" "Library:3mm5 Mono Aux" (at 177.8 45.72 0)
       (effects (font (size 1.27 1.27)) hide)
     )
@@
       (effects (font (size 1.27 1.27)) hide)
     )
-    (property "Footprint" "Library:aux_flush" (at 70.485 106.68 0)
+    (property "Footprint" "Library:3mm5 Mono Aux" (at 70.485 106.68 0)
       (effects (font (size 1.27 1.27)) hide)
     )
@@
       (effects (font (size 1.27 1.27)) hide)
     )
-    (property "Footprint" "Library:aux_flush" (at 88.9 76.2 0)
+    (property "Footprint" "Library:3mm5 Mono Aux" (at 88.9 76.2 0)
       (effects (font (size 1.27 1.27)) hide)
     )
@@
       (effects (font (size 1.27 1.27)) hide)
     )
-    (property "Footprint" "Library:aux_flush" (at 273.05 59.055 0)
+    (property "Footprint" "Library:3mm5 Mono Aux" (at 273.05 59.055 0)
       (effects (font (size 1.27 1.27)) hide)
     )
@@
       (effects (font (size 1.27 1.27)))
     )
-    (property "Footprint" "" (at 234.315 103.505 0)
+    (property "Footprint" "Package_DIP:DIP-14_W7.62mm_Socket" (at 234.315 103.505 0)
       (effects (font (size 1.27 1.27)) hide)
     )
@@
       (effects (font (size 1.27 1.27)))
     )
-    (property "Footprint" "" (at 214.63 59.055 0)
+    (property "Footprint" "Package_DIP:DIP-14_W7.62mm_Socket" (at 214.63 59.055 0)
       (effects (font (size 1.27 1.27)) hide)
     )
@@
       (effects (font (size 1.27 1.27)) hide)
     )
-    (property "Footprint" "Library:aux_flush" (at 176.53 111.76 0)
+    (property "Footprint" "Library:3mm5 Mono Aux" (at 176.53 111.76 0)
       (effects (font (size 1.27 1.27)) hide)
     )
@@
       (effects (font (size 1.27 1.27)) hide)
     )
-    (property "Footprint" "Library:aux_flush" (at 129.54 70.485 0)
+    (property "Footprint" "Library:3mm5 Mono Aux" (at 129.54 70.485 0)
       (effects (font (size 1.27 1.27)) hide)
     )
@@
       (effects (font (size 1.27 1.27)))
     )
-    (property "Footprint" "" (at 231.14 142.875 0)
+    (property "Footprint" "Package_DIP:DIP-14_W7.62mm_Socket" (at 231.14 142.875 0)
       (effects (font (size 1.27 1.27)) hide)
     )
@@
       (effects (font (size 1.27 1.27)) hide)
     )
-    (property "Footprint" "Library:aux_flush" (at 239.395 74.295 0)
-      (effects (font (size 1.27 1.27)) hide)
-    )
+    (property "Footprint" "Library:3mm5 Mono Aux" (at 239.395 74.295 0)
+      (effects (font (size 1.27 1.27)) hide)
+    )
