File: Bell/Bell.kicad_pcb (KiCad board)
At the start: 2 copper layers, 68.8 x 128.5 mm, 58 parts, among them J1 Conn_01x06_Female, J2 Conn_01x10_Pin, J3 Conn_01x10_Pin, Q1 BC547, Q11 BC557, Q12 BC547, Q13 BC547, Q14 BC547, Q15 BC547, Q2 BC557, Q3 BC557, Q4 BC547, Q5 BC547, U1 TL074, U10 Aux_flush, U2 Aux_flush, U3 TL072, U4 Aux_flush, U6 Aux_flush

Commit message: Add files via upload
Parts:
- added ?: , , F.Cu at (58.7, 45.5)
- added ?: , , F.Cu at (51.9, 132.0)
- added ?: , , F.Cu at (51.9, 114.0)
- added ?: , , F.Cu at (58.9, 90.6)
- added ?: , , F.Cu at (58.9, 68.2)
- added ?: , , F.Cu at (64.9, 114.0)
- added ?: , , F.Cu at (64.9, 132.0)
- U10, U2, U4, U6: footprint Library:aux_flush -> Library:3mm5 Mono Aux
- moved REF** 45.0 mm to (67.0, 147.5)
- moved REF** 45.0 mm to (67.0, 25.0)
- moved R13 16.6 mm to (106.7, 120.0), turned to 180 degrees
- moved D2 15.2 mm to (107.2, 122.8)
- turned U10 to -90 degrees
- turned U2 to -90 degrees
- turned U4 to -90 degrees
- turned U6 to -90 degrees
Routing:
- net Net-(R13-Pad1): track 3.08 -> 21.6 mm
- net ACC: track 98.9 -> 83.6 mm
- net OUT: track 110.9 -> 110.3 mm
- net IN2: track 73.3 -> 72.7 mm
- net Net-(R21-Pad1): track 34.1 -> 33.5 mm
Other:
- board size 68.8 x 128.5 mm -> 113.8 x 128.5 mm
