File: Bell/Bell.kicad_sch (KiCad schematic)
At the start: 56 parts, among them J1 Conn_01x06_Female, J2 Conn_01x10_Pin, J3 Conn_01x10_Pin, Q1 BC547, Q10 BC547, Q2 BC557, Q4 BC547, Q5 BC547, Q6 BC547, Q8 BC547, U1 Aux_flush, U1 TL074, U3 Aux_flush, U3 TL072

Commit message: Add files via upload
Parts:
- U1, U3: footprint Library:aux_flush -> Library:3mm5 Mono Aux
Changed lines of the file:
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@@
       (effects (font (size 1.27 1.27)) hide)
     )
-    (pin "2")
+    (pin "1")
+    (pin "10")
+    (pin "2")
+    (pin "3")
+    (pin "4")
+    (pin "5")
     (pin "6")
-    (pin "5")
+    (pin "7")
     (pin "8")
-    (pin "4")
     (pin "9")
-    (pin "3")
-    (pin "7")
-    (pin "10")
-    (pin "1")
     (instances
       (project "Bell"
@@
       (effects (font (size 1.27 1.27)) hide)
     )
-    (property "Footprint" "Library:aux_flush" (at 257.81 95.25 0)
+    (property "Footprint" "Library:3mm5 Mono Aux" (at 257.81 95.25 0)
       (effects (font (size 1.27 1.27)) hide)
     )
@@
       (effects (font (size 1.27 1.27)) hide)
     )
-    (pin "2")
-    (pin "1")
+    (pin "1")
+    (pin "2")
+    (pin "3")
+    (pin "5")
     (pin "6")
     (pin "7")
     (pin "4")
-    (pin "3")
     (pin "8")
-    (pin "5")
     (instances
       (project "Bell"
@@
       (effects (font (size 1.27 1.27)) hide)
     )
-    (property "Footprint" "Library:aux_flush" (at 22.86 161.29 0)
+    (property "Footprint" "Library:3mm5 Mono Aux" (at 22.86 161.29 0)
       (effects (font (size 1.27 1.27)) hide)
     )
@@
       (effects (font (size 1.27 1.27)) (justify left) hide)
     )
+    (pin "1")
+    (pin "2")
     (pin "3")
-    (pin "1")
-    (pin "2")
     (instances
       (project "Bells"
@@
       (effects (font (size 1.27 1.27)) hide)
     )
-    (pin "2")
-    (pin "1")
+    (pin "1")
+    (pin "2")
+    (pin "3")
+    (pin "5")
     (pin "6")
     (pin "7")
     (pin "4")
-    (pin "3")
     (pin "8")
-    (pin "5")
     (instances
       (project "Bell"
@@
       (effects (font (size 1.27 1.27)) hide)
     )
+    (pin "1")
+    (pin "2")
+    (pin "3")
     (pin "5")
+    (pin "6")
     (pin "7")
+    (pin "10")
     (pin "8")
+    (pin "9")
+    (pin "12")
+    (pin "13")
+    (pin "14")
     (pin "11")
-    (pin "3")
-    (pin "2")
-    (pin "1")
-    (pin "14")
-    (pin "6")
-    (pin "9")
-    (pin "13")
     (pin "4")
-    (pin "12")
-    (pin "10")
     (instances
       (project "Bell"
@@
       (effects (font (size 1.27 1.27)) hide)
     )
+    (pin "1")
+    (pin "2")
+    (pin "3")
     (pin "5")
+    (pin "6")
     (pin "7")
+    (pin "10")
     (pin "8")
+    (pin "9")
+    (pin "12")
+    (pin "13")
+    (pin "14")
     (pin "11")
-    (pin "3")
-    (pin "2")
-    (pin "1")
-    (pin "14")
-    (pin "6")
-    (pin "9")
-    (pin "13")
     (pin "4")
-    (pin "12")
-    (pin "10")
     (instances
       (project "Bell"
@@
       (effects (font (size 1.27 1.27)) hide)
     )
-    (property "Footprint" "Library:aux_flush" (at 154.94 151.892 0)
+    (property "Footprint" "Library:3mm5 Mono Aux" (at 154.94 151.892 0)
       (effects (font (size 1.27 1.27)) hide)
     )
@@
       (effects (font (size 1.27 1.27)) hide)
     )
+    (pin "1")
+    (pin "2")
+    (pin "3")
     (pin "5")
+    (pin "6")
     (pin "7")
+    (pin "10")
     (pin "8")
+    (pin "9")
+    (pin "12")
+    (pin "13")
+    (pin "14")
     (pin "11")
-    (pin "3")
-    (pin "2")
-    (pin "1")
-    (pin "14")
-    (pin "6")
-    (pin "9")
-    (pin "13")
     (pin "4")
-    (pin "12")
-    (pin "10")
     (instances
       (project "Bell"
@@
       (effects (font (size 1.27 1.27)) hide)
     )
-    (property "Footprint" "Library:aux_flush" (at 68.58 180.34 0)
+    (property "Footprint" "Library:3mm5 Mono Aux" (at 68.58 180.34 0)
       (effects (font (size 1.27 1.27)) hide)
     )
@@
       (effects (font (size 1.27 1.27)) (justify left) hide)
     )
+    (pin "1")
+    (pin "2")
     (pin "3")
-    (pin "1")
-    (pin "2")
     (instances
       (project "Bells"
@@
       (effects (font (size 1.27 1.27)) hide)
     )
+    (pin "1")
+    (pin "2")
+    (pin "3")
     (pin "5")
+    (pin "6")
     (pin "7")
+    (pin "10")
     (pin "8")
+    (pin "9")
+    (pin "12")
+    (pin "13")
+    (pin "14")
     (pin "11")
-    (pin "3")
-    (pin "2")
-    (pin "1")
-    (pin "14")
-    (pin "6")
-    (pin "9")
-    (pin "13")
     (pin "4")
-    (pin "12")
-    (pin "10")
     (instances
       (project "Bell"
@@
       (effects (font (size 1.27 1.27)) (justify left) hide)
     )
+    (pin "1")
+    (pin "2")
     (pin "3")
-    (pin "1")
-    (pin "2")
     (instances
       (project "Bells"
@@
       (effects (font (size 1.27 1.27)) hide)
     )
-    (pin "2")
-    (pin "1")
+    (pin "1")
+    (pin "2")
+    (pin "3")
+    (pin "5")
     (pin "6")
     (pin "7")
     (pin "4")
-    (pin "3")
     (pin "8")
-    (pin "5")
     (instances
       (project "Bell"
@@
       (effects (font (size 1.27 1.27)) (justify left) hide)
     )
+    (pin "1")
+    (pin "2")
     (pin "3")
-    (pin "1")
-    (pin "2")
     (instances
       (project "Bells"
@@
       (effects (font (size 1.27 1.27)) (justify left) hide)
     )
+    (pin "1")
+    (pin "2")
     (pin "3")
-    (pin "1")
-    (pin "2")
     (instances
       (project "Bells"
@@
       (effects (font (size 1.27 1.27)) hide)
     )
-    (pin "2")
+    (pin "1")
+    (pin "10")
+    (pin "2")
+    (pin "3")
+    (pin "4")
+    (pin "5")
     (pin "6")
-    (pin "5")
+    (pin "7")
     (pin "8")
-    (pin "4")
     (pin "9")
-    (pin "3")
-    (pin "7")
-    (pin "10")
-    (pin "1")
     (instances
       (project "Bell"
@@
       (effects (font (size 1.27 1.27)) hide)
     )
+    (pin "1")
+    (pin "2")
+    (pin "3")
     (pin "5")
+    (pin "6")
     (pin "7")
+    (pin "10")
     (pin "8")
+    (pin "9")
+    (pin "12")
+    (pin "13")
+    (pin "14")
     (pin "11")
-    (pin "3")
-    (pin "2")
-    (pin "1")
-    (pin "14")
-    (pin "6")
-    (pin "9")
-    (pin "13")
     (pin "4")
-    (pin "12")
-    (pin "10")
-    (instances
-      (project "Bell"
+    (instances
+      (project "Bell"
