File: LFO2/LFO2.kicad_sch (KiCad schematic)
At the start: 62 parts, among them J1 Conn_01x06_Female, J10 Conn_01x01_Pin, J11 Conn_01x01_Pin, J2 Conn_01x13_Pin, J3 Conn_01x13_Pin, J4 Conn_01x01_Pin, J5 Conn_01x01_Pin, J6 Conn_01x01_Pin, J7 Conn_01x01_Pin, J8 Conn_01x01_Pin, J9 Conn_01x01_Pin, Q1 BC547, Q1 BC557, Q3 BC557, SW1 SW_SPDT, SW2 SW_SPDT, U1 TL074, U2 Aux_flush, U2 DG417xJ, U4 TL072, U6 Aux_flush, U8 LM13700

Commit message: Add files via upload
Parts:
- added R15 (x4): 100k, Resistor_THT:R_Axial_DIN0204_L3.6mm_D1.6mm_P7.62mm_Horizontal, symbol Device:R
Connections:
- net +12V: now also R15.2
- net ABC: now also SW2.2 (B), U8.16
- net CAP: now also C2.1, SW1.1 (A), R15.2
- net CV2: now also Q3.1 (C), SW2.3 (C)
- net GND: now also R15.2
- net ITRI: now also R13.1, R15.1, U4.1
- net SQR: now also D4.1 (K), R13.1, R15.1, R15.2, R15.2
- net STOP: now also D3.2 (A), U2.1
- net SW: now also Q1.1 (C), SW1.2 (B), U1.9 (-), U2.8
- net TRI: now also R13.1, R15.2, U1.14, R15.1
- net VGND: now also R15.1, R15.1, R15.2, U1.2 (-)
- new net: R15.1, R15.1, U1.12 (+)
- new net: R15.1, R15.2, U1.13 (-)
Other:
- title: (none) -> LFO2 by github.com/Fihdi

Commit message: Add files via upload
Parts:
- removed J10, J11, J6, J7, J8, J9: Conn_01x01_Pin, Connector_PinHeader_2.54mm:PinHeader_1x01_P2.54mm_Vertical, symbol Connector:Conn_01x01_Pin
- removed R15 (x3): 100k, Resistor_THT:R_Axial_DIN0204_L3.6mm_D1.6mm_P7.62mm_Horizontal, symbol Device:R
- added R25, R28, R29: 100k, Resistor_THT:R_Axial_DIN0204_L3.6mm_D1.6mm_P7.62mm_Horizontal, symbol Device:R
- added R32: 4k7, Resistor_THT:R_Axial_DIN0204_L3.6mm_D1.6mm_P7.62mm_Horizontal, symbol Device:R
Connections:
- net +12V: now also R25.2; no longer U2.5 (VL)
- net CV2: no longer J4.1 (Pin_1), J5.1 (Pin_1)
- net GND: now also D2.2 (A), D4.2 (A), R28.2, R29.2, R32.1; no longer U4.3 (+)
- net SQR: now also U4.6 (-), U4.7; no longer D4.1 (K), R15.1, R15.2
- net SW: now also U1.12 (+)
- net TRI: now also U1.13 (-)
- net VGND: now also J4.1 (Pin_1), J5.1 (Pin_1)
- net at D1.1 (K), Q1.1 (C), U6.1: now also R32.2
- net at D2.1 (K), Q1.2 (B), R15.1: now also C2.2
- net at R15.1, R15.1: now also U4.3 (+); no longer U1.12 (+)
- net at R15.1, R15.2, U1.10 (+): now also D4.1 (K), U4.5 (+)
- net at U1.8: now also R15.1, R15.2; no longer D4.2 (A)
- net at C2.1, R16.1: now also R29.1
- net CAP: no longer names the net of C2.1, SW1.1 (A)
- net CAP: no longer J2.5 (Pin_5), J3.5 (Pin_5)
- new net: R25.1, R28.1, U2.5 (VL)
- no-connect marks 0 -> 2

Commit message: Add files via upload
Parts:
- added R33: 4k7, Resistor_THT:R_Axial_DIN0204_L3.6mm_D1.6mm_P7.62mm_Horizontal, symbol Device:R
- renumbered C2 to C1, C2 to C4, C1 to C6, Q1 to Q2, Q1 to Q4, R15 to R1, R15 to R10, R15 to R11, R15 to R12, R15 to R13, R16 to R14, R15 to R16, R15 to R17, R16 to R18, R13 to R19, R16 to R2, R16 to R20, R15 to R21, R15 to R22, R15 to R23, R15 to R24, R15 to R26, R16 to R27, R15 to R3, R15 to R30, R15 to R31, R13 to R4, R13 to R5, R18 to R6, R15 to R7, R15 to R8, R16 to R9, U2 to U12, U2 to U13, U6 to U15, U6 to U16, U6 to U3, U6 to U5, U2 to U9
Connections:
- net GND: now also R33.1
- net SQR: now also D1.2 (A)
- net at Q2.1 (C), R32.2, U3.1: now also R18.1; no longer D1.1 (K)
- new net: D1.1 (K), R33.2
Other:
- moved on the sheet: D1, R18
