File: RandomSource/RandomSource.kicad_sch (KiCad schematic)
At the start: 55 parts, among them J1 Conn_01x20_Pin, J2 Conn_01x06_Pin, J6 Conn_01x20_Pin, Q1 BC547, Q2 BC547, Q3 BC547, Q4 BC557, Q5 MMBFJ113, Q6 2N7000, U1 TL074, U10 Aux_flush, U11 Aux_flush, U13 Aux_flush, U14 Aux_flush, U2 Aux_flush, U3 Switch, U4 TL074, U5 Switch, U6 Aux_flush, U7 Switch, U8 Switch, U9 Aux_flush

Commit message: Add files via upload
Parts:
- removed D2: D, Diode_THT:D_A-405_P5.08mm_Vertical_AnodeUp, symbol Device:D
- removed Q5: MMBFJ113, Package_TO_SOT_THT:TO-92S_Wide, symbol Transistor_FET:MMBFJ113
- removed Q6: 2N7000, Package_TO_SOT_THT:TO-92L_Wide, symbol Transistor_FET:2N7000
- removed R13: 1k, Resistor_THT:R_Axial_DIN0204_L3.6mm_D1.6mm_P7.62mm_Horizontal, symbol Device:R
- removed R14, R19: 100k, Resistor_THT:R_Axial_DIN0204_L3.6mm_D1.6mm_P7.62mm_Horizontal, symbol Device:R
- removed R15: 1M, Resistor_THT:R_Axial_DIN0204_L3.6mm_D1.6mm_P7.62mm_Horizontal, symbol Device:R
- removed unit 2 of U1
- added C8: 100n, Capacitor_THT:C_Axial_L3.8mm_D2.6mm_P7.50mm_Horizontal, symbol Device:C
- added D5: D, Diode_THT:D_A-405_P5.08mm_Vertical_AnodeUp, symbol Device:D
- added R20: 10k, Resistor_THT:R_Axial_DIN0204_L3.6mm_D1.6mm_P7.62mm_Horizontal, symbol Device:R
- added R21, R22, R23, R24, R25: 1k, Resistor_THT:R_Axial_DIN0204_L3.6mm_D1.6mm_P7.62mm_Horizontal, symbol Device:R
- added U12: CD4066BE, Package_DIP:DIP-14_W7.62mm, symbol Analog_Switch:CD4066BE
Connections:
- net +12V: now also U12.14 (V_{DD})
- net BURST: now also R24.2, U12.3; no longer U9.1
- net COMPO: now also J1.17 (Pin_17), J6.17 (Pin_17), C8.2, R23.2, R25.2, U12.5; no longer J1.11 (Pin_11), J6.11 (Pin_11), U10.1
- net GATE: now also J1.11 (Pin_11), J6.11 (Pin_11), U12.4; no longer J1.17 (Pin_17), J6.17 (Pin_17)
- net GND: now also D3.2 (A), C8.1, D5.2 (A), U12.7 (V_{SS})
- net NOISE: now also R22.1; no longer U14.1
- net PULS: now also U12.13
- net SAH: now also R21.2; no longer U13.1
- net SHIN: now also R20.1; no longer U4.5 (+)
- net at U1.8: now also R25.1; no longer D3.2 (A)
- net at C5.2, U4.10 (+): now also U12.2
- net at U4.6 (-), U4.7: now also U12.1
- new net: D5.1 (K), R20.2, U4.5 (+)
- new net: R23.1, U10.1
- new net: R22.2, U14.1
- new net: R24.1, U9.1
- new net: R21.1, U13.1
Other:
- moved on the sheet: D4, J1, J6, RV1, RV2, RV3, U1C, U1D, U4A, U4B, U4C, U4D
