File: Mixer/Mixer.kicad_pcb (KiCad board)
At the start: 2 copper layers, 110.2 x 129 mm, 39 parts, among them J1 Conn_01x06_Male, Q1 BC547, Q2 BC557, U1 TL072, U2 Aux_flush, U3 Aux_flush, U4 Aux_flush, U5 Aux_flush, U6 Aux_flush

Commit message: Add files via upload
Parts:
- removed D2: LED, LED_THT:LED_D5.0mm
- removed Q2: BC557, Package_TO_SOT_THT:TO-92_Inline_Wide
- removed R12: 50k, Resistor_THT:R_Axial_DIN0204_L3.6mm_D1.6mm_P7.62mm_Horizontal
- added REF**: MountingHole_3.2mm_M3, MountingHole:MountingHole_3.2mm_M3, F.Cu at (100.0, 30.6)
- added REF**: MountingHole_3.2mm_M3, MountingHole:MountingHole_3.2mm_M3, F.Cu at (125.5, 153.1)
- added REF**: MountingHole_3.2mm_M3, MountingHole:MountingHole_3.2mm_M3, F.Cu at (125.4, 30.6)
- added REF**: MountingHole_3.2mm_M3, MountingHole:MountingHole_3.2mm_M3, F.Cu at (100.1, 153.1)
- moved R6 11.2 mm to (174.9, 43.2)
- moved R8 11.1 mm to (188.9, 43.5)
- moved R7 10.9 mm to (186.5, 51.1)
- moved U1 9.02 mm to (175.7, 46.5)
- moved D1 6.52 mm to (182.9, 139.2)
- moved J1 6.52 mm to (191.4, 83.8)
- moved Q1 6.52 mm to (173.1, 136.7)
- moved R1 6.52 mm to (159.5, 135.6)
- moved R10 6.52 mm to (185.7, 128.2)
- moved R11 6.52 mm to (178.1, 131.5)
- moved R13 6.52 mm to (186.0, 68.8)
- moved R14 6.52 mm to (159.7, 115.9)
- moved R15 6.52 mm to (159.7, 57.7)
- moved R16 6.52 mm to (159.7, 96.1)
- moved R17 6.52 mm to (159.7, 76.9)
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Routing:
- net Net-(D2-A): track 11.3 -> 0.00 mm
- net Net-(R10-Pad1): track 101.2 -> 94.6 mm
- net Net-(U1A--): track 104.6 -> 99.6 mm
- net -9V: track 148.6 -> 152.4 mm, vias 0 -> 1
- net Net-(Q2-E): track 3.10 -> 0.00 mm
- net Net-(U1B--): track 7.96 -> 5.92 mm
- net Net-(R6-Pad2): track 14.1 -> 12.3 mm
Other:
- board size 110.2 x 129 mm -> 101.6 x 129 mm
- board text added: "1"
- board text added: "2"
- board text added: "3"
- board text added: "4"
- board text added: "MIXΣR"
- board text removed: "MIXER"
