File: ClockDividerV2/ClockDividerV2.kicad_sch (KiCad schematic)
At the start: 65 parts, among them J1 Conn_01x06_Pin, J10 Conn_01x01_Pin, J2 Conn_01x14_Pin, J3 Conn_01x03_Pin, J4 Conn_01x14_Pin, J5 Conn_01x01_Pin, J6 Conn_01x01_Pin, J7 Conn_01x01_Pin, J8 Conn_01x01_Pin, J9 Conn_01x01_Pin, Q1 BC547, Q2 BC547, Q3 BC547, Q4 BC547, Q5 BC557, SW1 SW_Push, SW2 SW_Push, SW3 SW_Push, U1 L7805, U10 Aux_flush, U11 Aux_flush, U12 Aux_flush, U2 ATmega328P-P, U4 Aux_flush, U5 Aux_flush, U6 Aux_flush, U7 TL074, U8 Aux_flush, U9 Aux_flush, Y1 Crystal

Commit message: Add files via upload
Parts:
- C1: value C -> 100n
- C2, C3: value C -> 22p
- R1, R14, R2, R20, R3, R4, R5, R6, R7, R8, R9: value R -> 10k
- R10, R11, R12, R13, R19: value R -> 2k2
- R15, R16, R17, R18: value R -> 1k
- R21: value R -> 100k
- R23, R24: value R -> 47k
- Y1: value Crystal -> 16MHz
